File: static/tools/tester/Testeur_new.brd (EAGLE design)
At the start: 101.6 x 108 mm, 35 parts, among them IC1 MEGA8-P, Q2 MFR475V

Commit message: [Tester] new design.
Parts:
- removed ALIM: (no value), pinhead:1X02
- removed C1-CRYSTAL, C2-CRYSTAL: 20 pF, capacitor-wima:C5B5
- removed C1-REGULATOR, C1-REGULATOR1, C2-REGULATOR, C2-REGULATOR1: (no value), capacitor-wima:C5B5
- removed ENCODER-IHM: CI-11, piher:CI-11
- removed IC2, IC3: (no value), v-reg:78XXS
- removed JP1, JP2: (no value), pinhead:2X12
- removed JP3: (no value), pinhead:1X16
- removed Q1: (no value), special:QS
- removed R6: (no value), rcl:0204/7
- removed SERVO-IHM, SERVO-IHM1, SERVO-IHM2: (no value), con-lstb:MA03-1
- removed SWITCH_5V: (no value), pinhead:1X03
- removed X1: (no value), con-wago-500:W237-102
- added 0->3, 10->13, A0->A3: (no value), pinhead:1X04
- added C1, C2: (no value), capacitor-wima:C5B3.5
- added ENCODER: CI-11, piher:CI-11
- added I²C: (no value), pinhead:1X02
- added LCD: (no value), pinhead:1X16
- added LCD_WIRES: (no value), pinhead:1X06
- added PWM, SWITCH, SWITCH1: (no value), pinhead:1X03
- added SERVO1, SERVO2: (no value), con-lstb:MA03-1
- added X2: (no value), con-wago-500:W237-102
- IC1: value MEGA8-P -> (none); device atmel:DIL28-3 -> v-reg:78XXS
- R3, R4: device resistor:0204/7 -> rcl:0204/7
- moved R1 83.8 mm to (-31.1, -46.4), turned to 180 degrees
- moved IC1 80.4 mm to (-92.1, -41.9), turned to 90 degrees
- moved R3 68.3 mm to (-31.1, -48.9), turned to 180 degrees
- moved RETURN_IHM 65.5 mm to (-17.8, -31.8), turned to 180 degrees
- moved R5 51.5 mm to (-20.3, -21.6), turned to 180 degrees
- moved R4 44.7 mm to (-20.3, -18.4), turned to 0 degrees
- moved R2 43.8 mm to (-31.1, -51.4)
- moved LED1 39.9 mm to (-43.8, -40.6)
- moved LED2 39.9 mm to (-43.8, -47.0)
- moved Q2 11.3 mm to (-57.1, -52.1), turned to 180 degrees
- moved MOTOR 6.54 mm to (-70.5, -48.3), turned to 0 degrees
- moved AR 3.59 mm to (-16.5, -12.7), turned to 270 degrees
- moved CODER-IHM 2.62 mm to (-64.8, -14.6), turned to 270 degrees
- moved I2C-IHM 2.62 mm to (-76.8, -14.6), turned to 270 degrees
- moved POTAR 2.01 mm to (-83.8, -30.5)
Connections:
- removed net 5V_P/A: SERVO-IHM.2, SERVO-IHM1.2, SERVO-IHM2.2, SWITCH_5V.2
- removed net 5V_POW_IHM: JP2.3
- removed net ENCODER1: IC1.6, JP1.24
- removed net ENCODER2: IC1.11, JP1.23
- removed net GND_IHM: AR.1, C1-REGULATOR1.2, C2-REGULATOR1.2, CODER-IHM.2, ENCODER-IHM.B, ENCODER-IHM.D, I2C-IHM.2, IC3.GND, JP2.1, JP3.1, JP3.10, JP3.5, JP3.7, JP3.8, JP3.9, LED1.K, LED2.K, POTAR.3, Q2.E, RETURN_IHM.1, SERVO-IHM.1, SERVO-IHM1.1, SERVO-IHM2.1, X1.2
- removed net INT_ODO1: IC1.4, JP1.18
- removed net LCD1: IC1.13, JP1.19
- removed net LCD2: IC1.14, JP1.17
- removed net LCD3: IC1.15, JP1.15
- removed net LCD5: IC1.18, JP1.9
- removed net LCD6: IC1.19, JP1.7
- removed net LED1: IC1.24, R4.1
- removed net LED2: IC1.25, R3.1
- removed net N$27: JP2.15, JP3.11
- removed net N$28: JP1.4, R4.2
- removed net N$29: JP2.13, JP3.12
- removed net N$30: JP2.9, JP3.13
- removed net N$34: JP2.7, JP3.14
- removed net N$35: JP2.11, R2.1, SERVO-IHM.3
- removed net N$36: JP2.8, RETURN_IHM.2
- removed net N$46: IC1.23, R5.1, R6.2
- removed net N$7: JP1.6, R3.2
- removed net RETURN: IC1.26, JP1.8
- removed net SCL: IC1.28, JP1.12
- removed net SDA: IC1.27, JP1.10
- removed net SELECT: IC1.12, JP1.21
- removed net SENS_ODO: IC1.5, JP1.22
- removed net SERVO/PWM: IC1.17, JP1.11
- removed net SERVO2: IC1.2, JP1.14
- removed net SERVO3: IC1.3, JP1.16
- removed net VCC: C2-REGULATOR.1, IC1.20, IC1.7, IC2.OUT, JP1.5, R1.1
- removed net VCC_IHM: CODER-IHM.1, I2C-IHM.1, JP2.5, JP3.2, POTAR.2, SWITCH_5V.1
- new net 5V_ARDUINO: CODER-IHM.1, I2C-IHM.1, LCD.2, POTAR.2, SWITCH.3
- new net 5V_EXT: C2.1, IC1.OUT, SWITCH.1
- new net N$15: 10->13.3, PWM.3, R2.1
- new net N$24: AR.2, R4.2
- new net N$5: A0->A3.2, ENCODER.C
- new net POWER: PWM.2, SERVO1.2, SERVO2.2, SWITCH1.2
- net 5V_POWER: now also SWITCH.2, SWITCH1.1; no longer C2-REGULATOR1.1, IC3.OUT, SWITCH_5V.3
- net ALIM_EXT: now also C1.1, IC1.IN, SWITCH1.3, X2.1; no longer C1-REGULATOR1.1, IC3.IN, X1.1
- net GND: now also AR.1, C1.2, C2.2, CODER-IHM.2, ENCODER.B, ENCODER.D, I2C-IHM.2, IC1.GND, LCD.1, LCD.10, LCD.5, LCD.7, LCD.8, LCD.9, LED1.K, LED2.K, POTAR.3, PWM.1, Q2.E, R5.1, RETURN_IHM.1, SERVO1.1, SERVO2.1, X2.2; no longer ALIM.1, C1-CRYSTAL.1, C1-REGULATOR.2, C2-CRYSTAL.1, C2-REGULATOR.2, IC1.22, IC1.8, IC2.GND, JP1.1, R5.2
- net N$1: now also A0->A3.3, RETURN_IHM.2; no longer C1-CRYSTAL.2, IC1.9, Q1.1
- net N$10: now also I²C.2; no longer JP2.10
- net N$11: now also I²C.1; no longer JP2.12
- net N$12: now also R1.2; no longer JP2.4
- net N$13: now also 10->13.4, ENCODER.E; no longer JP2.6, LED2.A
- net N$14: now also 0->3.4, SERVO1.3; no longer JP2.14, SERVO-IHM1.3
- net N$16: now also 0->3.2; no longer JP2.18
- net N$17: now also 0->3.1; no longer JP2.22
- net N$18: now also A0->A3.1, ENCODER.A; no longer ENCODER-IHM.A, JP2.24
- net N$2: now also LCD.11, LCD_WIRES.4; no longer C2-CRYSTAL.2, IC1.10, Q1.2
- net N$21: now also 10->13.2, R1.1; no longer ENCODER-IHM.C, JP2.23
- net N$22: now also 10->13.1, R3.1; no longer ENCODER-IHM.E, JP2.21
- net N$25: now also LCD.4, LCD_WIRES.6; no longer JP2.19, JP3.4
- net N$26: now also LCD.6, LCD_WIRES.5; no longer JP2.17, JP3.6
- net N$3: now also LCD.12, LCD_WIRES.3; no longer JP1.2, R6.1
- net N$37: now also A0->A3.4, R4.1, R5.2; no longer AR.2, JP2.2
- net N$39: now also LCD.3; no longer JP3.3
- net N$4: now also LCD.13, LCD_WIRES.2; no longer IC1.1, R1.2
- net N$42: now also 0->3.3, SERVO2.3; no longer JP2.16, SERVO-IHM2.3
- net N$6: now also LCD.14, LCD_WIRES.1; no longer ALIM.2, C1-REGULATOR.1, IC2.IN
- net N$9: now also LED2.A, R3.2; no longer IC1.16, JP1.13
Routing:
- net GND_IHM: track 290.9 -> 0.00 mm, vias 1 -> 0
- net GND: track 93.4 -> 251.5 mm
- net ENCODER1: track 96.6 -> 0.00 mm
- net N$17: track 101.5 -> 7.77 mm, vias 2 -> 0
- net SENS_ODO: track 87.7 -> 0.00 mm, vias 1 -> 0
- net N$21: track 92.2 -> 8.78 mm
- net VCC_IHM: track 83.4 -> 0.00 mm, vias 4 -> 0
- net N$16: track 90.7 -> 12.1 mm, vias 2 -> 0
- net N$11: track 79.2 -> 5.71 mm
- net N$22: track 77.5 -> 4.45 mm
- net INT_ODO1: track 72.0 -> 0.00 mm
- net N$10: track 71.7 -> 5.71 mm
- net VCC: track 62.3 -> 0.00 mm
- net SERVO3: track 60.0 -> 0.00 mm
- net 5V_ARDUINO: track 0.00 -> 59.3 mm
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Other:
- board size 101.6 x 108 mm -> 101.6 x 52.1 mm
- board text removed: "A"
- board text removed: "AR"
- board text removed: "B"
- board text removed: "BOTTOM"
- board text removed: "GND"
- board text removed: "I²C"
- board text removed: "LED1"
- board text removed: "LED2"
- board text removed: "MOTOR"
- board text removed: "POWER"
- board text removed: "TOP"
- board text removed: "battery"
- board text removed: "by Fab@ENAC - 2015"
- board text removed: "coder"
- board text removed: "encoder"
- board text removed: "potar"
- board text removed: "return"
- board text removed: "servo1"
- board text removed: "servo2"
- board text removed: "servo3"
