File: primary_robot/aiio/IA-prop-raspberry.brd (EAGLE design)
At the start: 116 x 156 mm, 60 parts, among them U1 ARDUINO_R3_SHIELD

Commit message: [AIIO] Adds a reset button for the Raspi
Parts:
- added PWR_RP2: (no value), SparkFun:TACTILE-PTH
Connections:
- new net RP2_PWR: PWR_RP2.2, RP2.26
- net GND: now also PWR_RP2.4
Changed lines of the file:
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@@
 <element name="R17" library="SparkFun" package="AXIAL-0.3" value="10K" x="-124.46" y="-40.64"/>
 <element name="R18" library="SparkFun" package="AXIAL-0.3" value="10K" x="-124.46" y="-45.72"/>
+<element name="PWR_RP2" library="SparkFun" package="TACTILE-PTH" value="" x="-137.16" y="-43.18"/>
 </elements>
 <signals>
@@
 <wire x1="10.16" y1="36.83" x2="8.89" y2="38.1" width="0.8128" layer="16"/>
 <wire x1="11.43" y1="38.1" x2="8.89" y2="38.1" width="0.8128" layer="16"/>
-<wire x1="55.88" y1="68.58" x2="53.34" y2="105.41" width="0" layer="19" extent="1-1"/>
-<wire x1="53.34" y1="49.53" x2="55.88" y2="68.58" width="0" layer="19" extent="1-1"/>
-<wire x1="45.72" y1="21.59" x2="53.34" y2="49.53" width="0" layer="19" extent="1-1"/>
-<wire x1="-8.475" y1="25.7778" x2="10.16" y2="27.94" width="0" layer="19" extent="1-16"/>
-<wire x1="-9.125" y1="25.7778" x2="-8.475" y2="25.7778" width="0" layer="19" extent="1-1"/>
-<wire x1="-9.775" y1="25.7778" x2="-9.125" y2="25.7778" width="0" layer="19" extent="1-1"/>
-<wire x1="-10.425" y1="25.7778" x2="-9.775" y2="25.7778" width="0" layer="19" extent="1-1"/>
-<wire x1="-11.075" y1="25.7778" x2="-10.425" y2="25.7778" width="0" layer="19" extent="1-1"/>
+<contactref element="PWR_RP2" pad="4"/>
+<wire x1="-53.34" y1="0" x2="-133.9088" y2="-45.4406" width="0" layer="19" extent="16-16"/>
+<wire x1="-16.925" y1="25.7778" x2="-20.32" y2="25.4" width="0" layer="19" extent="1-16"/>
+<wire x1="-11.075" y1="25.7778" x2="-16.925" y2="25.7778" width="0" layer="19" extent="1-1"/>
+<wire x1="-10.425" y1="25.7778" x2="-11.075" y2="25.7778" width="0" layer="19" extent="1-1"/>
+<wire x1="-9.775" y1="25.7778" x2="-10.425" y2="25.7778" width="0" layer="19" extent="1-1"/>
+<wire x1="-9.125" y1="25.7778" x2="-9.775" y2="25.7778" width="0" layer="19" extent="1-1"/>
+<wire x1="-8.475" y1="25.7778" x2="-9.125" y2="25.7778" width="0" layer="19" extent="1-1"/>
 <wire x1="-11.075" y1="19.9422" x2="-11.075" y2="25.7778" width="0" layer="19" extent="1-1"/>
-<wire x1="-16.925" y1="25.7778" x2="-11.075" y2="25.7778" width="0" layer="19" extent="1-1"/>
-<wire x1="-20.32" y1="25.4" x2="-16.925" y2="25.7778" width="0" layer="19" extent="1-16"/>
+<wire x1="10.16" y1="27.94" x2="-8.475" y2="25.7778" width="0" layer="19" extent="1-16"/>
 <wire x1="-31.75" y1="60.96" x2="-35.56" y2="38.1" width="0" layer="19" extent="1-1"/>
 <wire x1="16.51" y1="60.96" x2="11.43" y2="38.1" width="0" layer="19" extent="1-1"/>
 <wire x1="15.76" y1="86.946" x2="16.51" y2="60.96" width="0" layer="19" extent="1-1"/>
 <wire x1="-21.59" y1="106.68" x2="-25.4" y2="80.296" width="0" layer="19" extent="1-1"/>
+<wire x1="53.34" y1="49.53" x2="45.72" y2="21.59" width="0" layer="19" extent="1-1"/>
+<wire x1="55.88" y1="68.58" x2="53.34" y2="49.53" width="0" layer="19" extent="1-1"/>
+<wire x1="53.34" y1="105.41" x2="55.88" y2="68.58" width="0" layer="19" extent="1-1"/>
 </signal>
 <signal name="N$4">
@@
 <signal name="N$50">
 </signal>
+<signal name="RP2_PWR">
+<contactref element="RP2" pad="26"/>
+<contactref element="PWR_RP2" pad="2"/>
+<wire x1="-9.64" y1="86.946" x2="-133.9088" y2="-40.9194" width="0" layer="19" extent="1-1"/>
+</signal>
 </signals>

Commit message: [AIIO_board] Add I2C bus "I2C0" for sonar sensors on shematic file.
Parts:
- added SV1, SV10, SV11, SV12, SV2, SV3, SV4, SV5, SV6, SV7, SV8, SV9: (no value), con-lsta:FE05-1
Connections:
- new net 5V: SV1.5, SV10.5, SV12.5, SV2.5, SV3.5, SV4.5, SV5.5, SV6.5, SV7.5, SV8.5, SV9.5
- new net I2C0_MODE: SV1.2, SV10.2, SV12.2, SV2.2, SV3.2, SV4.2, SV5.2, SV6.2, SV7.2, SV8.2, SV9.2
- new net I2C0_SCL: SV1.3, SV10.3, SV12.3, SV2.3, SV3.3, SV4.3, SV5.3, SV6.3, SV7.3, SV8.3, SV9.3
- new net I2C0_SDA: SV1.4, SV10.4, SV12.4, SV2.4, SV3.4, SV4.4, SV5.4, SV6.4, SV7.4, SV8.4, SV9.4
- net GND: now also SV1.1, SV10.1, SV12.1, SV2.1, SV3.1, SV4.1, SV5.1, SV6.1, SV7.1, SV8.1, SV9.1
