File: 2016/primary/aiio/IA-prop-raspberry.brd (EAGLE design)
At the start: 0.3 x 0.3 mm, 74 parts, among them U1 ARDUINO_R3_SHIELD

Commit message: [AIIO_boards] Create and add components for IHM_BOARD.
Parts:
- added 12V_BOARDS, 12V_BOARDS_SRC, 12V_PROPU_SRC: (no value), con-ptr500:AK300/2
- added BOARDIHM_CON_IHM: (no value), con-lsta:FE06
- added LED4, LED5: (no value), adafruit:LED5MM
- added LED6: RGBLED_CA-5MM, adafruit:LED5MMRGB
- added R19, R20: 680, SparkFun:AXIAL-0.3
- added U$10: CORD, club:CORD
- added U$4: BAU, club:BAU_30
- added U$5: FUSE, club:FUSE_PROPU
- added U$6, U$8: SWITCH_01, club:SWITCH_01
- added U$7: FUSE_BOARDS, club:FUSE_BOARDS
- added U$9: PUSH_BUT_COL_SELEC, club:PUSH_BUT_COL_SELEC
- moved BAT_12V_BOARDS 215.0 mm to (-170.2, -127.0), turned to 0 degrees
Connections:
- new net BAT_12V_BOARDS+: BAT_12V_BOARDS.1, U$7.P$1
- new net BAT_12V_BOARDS-: 12V_BOARDS_SRC.2, BAT_12V_BOARDS.2, R20.P$2
- new net BAT_12V_PROPU+: BAT_12V_PROPU.1, U$4.P1
- new net BAT_12V_PROPU-: 12V_PROPU_SRC.2, BAT_12V_PROPU.2, R19.P$2
- new net BOARDIHM_GND: BOARDIHM_CON_IHM.3, LED6.2, U$10.P$2
- new net N$10: U$5.P$2, U$6.P$1
- new net N$11: 12V_PROPU_SRC.1, LED4.A, U$6.P$2
- new net N$12: LED4.K, R19.P$1
- new net N$13: U$7.P$2, U$8.P$1
- new net N$14: 12V_BOARDS_SRC.1, LED5.A, U$8.P$2
- new net N$15: BOARDIHM_CON_IHM.2, LED6.1
- new net N$16: LED5.K, R20.P$1
- new net N$18: BOARDIHM_CON_IHM.4, U$10.P$1
- new net N$51: BOARDIHM_CON_IHM.5, LED6.3
- new net N$52: BOARDIHM_CON_IHM.6, LED6.4
- new net N$6: BOARDIHM_CON_IHM.1, U$9.P$1
- new net N$8: U$4.P2, U$5.P$1
- net +12V: now also 12V_BOARDS.1; no longer BAT_12V_BOARDS.1
- net GND_12: now also 12V_BOARDS.2; no longer BAT_12V_BOARDS.2

Commit message: [AIIO_boards] Clean schematic and board files.
Parts:
- added 12V_BOARDS_SRC1, 12V_PROPU_SRC1: (no value), con-ptr500:AK300/2
- added U$11: FOOTPRINT_PRIMAIRE2016, footprintPrimaire2016:PRIMAIRE2016
- moved U$10 610.5 mm to (370.8, -81.3), turned to 180 degrees
- moved U$9 605.7 mm to (387.4, -82.5)
- moved BOARDIHM_CON_IHM 598.9 mm to (387.4, -99.1), turned to 270 degrees
- moved U$4 588.8 mm to (421.6, -39.4)
- moved LED6 584.4 mm to (358.1, -102.9)
- moved U$5 584.1 mm to (411.5, -62.2), turned to 180 degrees
- moved 12V_PROPU_SRC 553.2 mm to (350.5, -39.4)
- moved U$6 550.7 mm to (360.7, -67.3)
- moved R19 548.0 mm to (342.9, -52.1)
- moved BAT_12V_PROPU 540.6 mm to (386.1, -39.4)
- moved LED4 540.2 mm to (331.5, -39.4)
- moved U$8 528.5 mm to (315.0, -69.8)
- moved LED5 527.8 mm to (320.0, -85.1)
- moved R20 516.9 mm to (311.1, -95.2), turned to 180 degrees
- moved 12V_BOARDS_SRC 509.7 mm to (292.1, -86.4)
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- renumbered X3 to 12V_BOARDS1
Connections:
- net BAT_12V_BOARDS-: now also 12V_BOARDS_SRC1.2
- net BAT_12V_PROPU-: now also 12V_PROPU_SRC1.2
- net BOARDIHM_GND: now also U$9.P$2
- net N$11: now also 12V_PROPU_SRC1.1
- net N$14: now also 12V_BOARDS_SRC1.1
- net N$39: now also R10.P$2
- net N$49: now also U1.D12

Commit message: [AIIO_board]Place connectors for sonar connectors.
Parts:
- added SV4-1: (no value), con-lsta:FE05-1
- moved SV11 1621.7 mm to (1177.8, 829.1), turned to 135 degrees
- moved SV10 1599.6 mm to (1126.1, 868.4), turned to 165 degrees
- moved SV12 1593.7 mm to (1181.3, 768.1), turned to 105 degrees
- moved RST_RP2 1555.3 mm to (1297.0, 929.8), turned to 60 degrees
- moved R2 1538.9 mm to (1290.0, 917.7), turned to 60 degrees
- moved LED3 1531.6 mm to (1287.7, 926.4), turned to 330 degrees
- moved SV9 1525.6 mm to (1069.2, 828.6), turned to 195 degrees
- moved SV1 1524.8 mm to (1182.5, 721.7), turned to 75 degrees
- moved SV2 1498.6 mm to (1185.3, 655.9), turned to 45 degrees
- moved RP2 1477.6 mm to (1281.3, 925.4), turned to 210 degrees
- moved SV8 1474.7 mm to (1028.9, 805.1), turned to 225 degrees
- moved U$7 1465.7 mm to (1498.0, 792.4), turned to 330 degrees
- moved BAT_12V_BOARDS 1459.6 mm to (1485.0, 774.9), turned to 330 degrees
- moved 12V_PROPU_SRC1 1456.6 mm to (1519.6, 781.4), turned to 330 degrees
- moved LED4 1452.9 mm to (1532.5, 778.3), turned to 330 degrees
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Connections:
- removed net 5V: SV1.5, SV10.5, SV12.5, SV2.5, SV3.5, SV4.5, SV5.5, SV6.5, SV7.5, SV8.5, SV9.5
- removed net MODE_SONAR: SV1.2, SV10.2, SV12.2, SV2.2, SV3.2, SV4.2, SV5.2, SV6.2, SV7.2, SV8.2, SV9.2
- removed net SCL_SONAR: SV1.3, SV10.3, SV12.3, SV2.3, SV3.3, SV4.3, SV5.3, SV6.3, SV7.3, SV8.3, SV9.3
- removed net SDA_SONAR: SV1.4, SV10.4, SV12.4, SV2.4, SV3.4, SV4.4, SV5.4, SV6.4, SV7.4, SV8.4, SV9.4
- new net 5V1: SV1.5, SV10.5, SV12.5, SV2.5, SV3.5, SV4-1.5, SV4.5, SV5.5, SV6.5, SV7.5, SV8.5, SV9.5
- new net GND1: SV1.1, SV10.1, SV12.1, SV2.1, SV3.1, SV4-1.1, SV4.1, SV5.1, SV6.1, SV7.1, SV8.1, SV9.1
- new net MODE_SONAR1: SV1.2, SV10.2, SV12.2, SV2.2, SV3.2, SV4-1.2, SV4.2, SV5.2, SV6.2, SV7.2, SV8.2, SV9.2
- new net SCL_SONAR1: SV1.3, SV10.3, SV12.3, SV2.3, SV3.3, SV4-1.3, SV4.3, SV5.3, SV6.3, SV7.3, SV8.3, SV9.3
- new net SDA_SONAR1: SV1.4, SV10.4, SV12.4, SV2.4, SV3.4, SV4-1.4, SV4.4, SV5.4, SV6.4, SV7.4, SV8.4, SV9.4
- net GND: no longer SV1.1, SV10.1, SV12.1, SV2.1, SV3.1, SV4.1, SV5.1, SV6.1, SV7.1, SV8.1, SV9.1
Routing:
- net 5V_PRP: track 89.1 -> 71.1 mm
- net GND: track 328.9 -> 326.4 mm
- net N$7: track 2.54 -> 5.08 mm
Other:
- board outline removed
- board text added: "SRV9"

Commit message: [AIIO_board]Place RP2 and make corrections on I2C_RP2 bus.
Parts:
- removed SV4-1: (no value), con-lsta:FE05-1
- added SV9-1: (no value), con-lsta:FE05-1
- moved RP2 139.0 mm to (1170.7, 841.2), turned to 180 degrees
Connections:
- removed net 5V1: SV1.5, SV10.5, SV12.5, SV2.5, SV3.5, SV4-1.5, SV4.5, SV5.5, SV6.5, SV7.5, SV8.5, SV9.5
- removed net GND1: SV1.1, SV10.1, SV12.1, SV2.1, SV3.1, SV4-1.1, SV4.1, SV5.1, SV6.1, SV7.1, SV8.1, SV9.1
- removed net MODE_SONAR1: SV1.2, SV10.2, SV12.2, SV2.2, SV3.2, SV4-1.2, SV4.2, SV5.2, SV6.2, SV7.2, SV8.2, SV9.2
- removed net SCL_SONAR1: SV1.3, SV10.3, SV12.3, SV2.3, SV3.3, SV4-1.3, SV4.3, SV5.3, SV6.3, SV7.3, SV8.3, SV9.3
- removed net SDA_SONAR1: SV1.4, SV10.4, SV12.4, SV2.4, SV3.4, SV4-1.4, SV4.4, SV5.4, SV6.4, SV7.4, SV8.4, SV9.4
- new net SCL_RP2: RP2.5, SV1.3, SV10.3, SV12.3, SV2.3, SV3.3, SV4.3, SV5.3, SV6.3, SV7.3, SV8.3, SV9-1.3, SV9.3
- new net SDA_RP2: RP2.3, SV1.4, SV10.4, SV12.4, SV2.4, SV3.4, SV4.4, SV5.4, SV6.4, SV7.4, SV8.4, SV9-1.4, SV9.4
- net 5V_PRP: now also SV1.5, SV10.5, SV12.5, SV2.5, SV3.5, SV4.5, SV5.5, SV6.5, SV7.5, SV8.5, SV9-1.5, SV9.5
- net GND: now also SV1.1, SV10.1, SV12.1, SV2.1, SV3.1, SV4.1, SV5.1, SV6.1, SV7.1, SV8.1, SV9-1.1, SV9.1

Commit message: [AIIO_boards] Connect servo connectors to PCA9685PW.
Parts:
- moved PWR_RP2 257.5 mm to (1099.1, 850.1)
- moved SRV15 154.9 mm to (1046.2, 684.0)
- moved SRV3 150.2 mm to (1069.2, 724.8)
- moved SRV11 148.7 mm to (1054.2, 698.2), turned to 240 degrees
- moved SRV6 144.0 mm to (1071.2, 707.4), turned to 240 degrees
- moved SRV7 143.5 mm to (1062.3, 711.9), turned to 240 degrees
- moved SRV14 143.1 mm to (1054.4, 678.8)
- moved SRV10 142.5 mm to (1063.0, 693.1), turned to 240 degrees
- moved CON_I2C_UART 141.3 mm to (1159.6, 661.3)
- moved P-UP_SCL 139.6 mm to (1155.7, 649.9)
- moved SRV9 139.0 mm to (1071.2, 688.4), turned to 240 degrees
- moved SRV8 138.3 mm to (1080.6, 683.0), turned to 240 degrees
- moved R7 138.3 mm to (1144.9, 637.0)
- moved P-UP_SDA 137.9 mm to (1151.7, 644.5)
- moved R4 137.5 mm to (1147.1, 640.7)
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Connections:
- net PWM12: now also U$1.22; no longer U$1.19
- net PWM13: now also U$1.21; no longer U$1.20
- net PWM14: now also U$1.20; no longer U$1.21
- net PWM15: now also U$1.19; no longer U$1.22
Routing:
- net SCL_RP2: track 0.00 -> 341.8 mm
- net SDA_RP2: track 0.00 -> 328.5 mm
- net GND: track 326.4 -> 635.9 mm, vias 0 -> 1
- net 5V_PRP: track 71.1 -> 325.8 mm
- net PWM3: track 0.00 -> 61.3 mm, vias 0 -> 1
- net PWM15: track 0.00 -> 59.1 mm, vias 0 -> 1
- net PWM11: track 0.00 -> 57.7 mm, vias 0 -> 1
- net PWM7: track 0.00 -> 55.7 mm, vias 0 -> 1
- net PWM2: track 0.00 -> 52.9 mm, vias 0 -> 1
- net PWM14: track 0.00 -> 51.4 mm, vias 0 -> 1
- net PWM6: track 0.00 -> 46.4 mm, vias 0 -> 1
- net PWM10: track 0.00 -> 45.4 mm, vias 0 -> 1
- net PWM1: track 0.00 -> 44.4 mm, vias 0 -> 1
- net PWM13: track 0.00 -> 42.9 mm, vias 0 -> 1
- net PWM5: track 0.00 -> 37.7 mm, vias 0 -> 1
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
Commit message: [AIIO_board] Make route for sonar I2C
Parts:
- moved R2 209.9 mm to (1097.0, 835.2), turned to 90 degrees
- moved LED3 206.4 mm to (1098.1, 844.7), turned to 150 degrees
- moved RST_RP2 204.5 mm to (1109.5, 848.2), turned to 180 degrees
- moved R12 169.8 mm to (1030.4, 703.5), turned to 240 degrees
- moved R13 150.8 mm to (1038.1, 699.4), turned to 240 degrees
- moved R10 149.1 mm to (1034.7, 705.2), turned to 240 degrees
- moved R11 146.3 mm to (1023.3, 699.3)
- moved LED1 84.6 mm to (1152.1, 590.7), turned to 240 degrees
- moved R9 82.0 mm to (1038.6, 707.0), turned to 240 degrees
- moved R8 76.0 mm to (1027.5, 708.6), turned to 240 degrees
- moved R3 64.6 mm to (1147.0, 581.9), turned to 240 degrees
- moved IHM 36.4 mm to (1039.0, 715.7), turned to 330 degrees
- moved R17 31.0 mm to (979.4, 674.7), turned to 60 degrees
- moved R16 28.5 mm to (982.4, 673.0), turned to 60 degrees
- moved R14 22.0 mm to (988.3, 669.9), turned to 60 degrees
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Connections:
- net 5V_PRP: now also SV11.5
- net GND: now also SV11.1
- net SCL_RP2: now also SV11.3
- net SDA_RP2: now also SV11.4
Routing:
- net 5V_PRP: track 325.8 -> 828.2 mm, vias 0 -> 2
- net SDA_RP2: track 328.5 -> 830.6 mm, vias 0 -> 2
- net SCL_RP2: track 341.8 -> 843.3 mm, vias 0 -> 2
- net GND: track 635.9 -> 1067.3 mm, vias 1 -> 3
- net RP2_PWR: track 0.00 -> 97.4 mm
- net N$1: track 0.00 -> 89.8 mm
- net N$42: track 0.00 -> 87.6 mm
- net N$48: track 0.00 -> 85.1 mm
- net N$46: track 0.00 -> 22.0 mm
- net N$47: track 0.00 -> 11.1 mm
- net N$49: track 0.00 -> 10.9 mm
- net N$44: track 0.00 -> 8.07 mm
- net N$43: track 0.00 -> 7.45 mm
- net N$3: track 0.00 -> 6.38 mm
- net N$41: track 0.00 -> 3.96 mm

Commit message: [AIIO_board] Update pin Ardu
Connections:
- removed net N$40: R9.P$2, U1.D6
- new net N$17: R9.P$2, U1.D3
- net N$45: now also U1.D6; no longer U1.D9
- net N$46: now also U1.D7; no longer U1.D3
- net N$47: now also U1.D4; no longer U1.D2
- net N$49: now also U1.D2; no longer U1.D12
- net PRESENCE_1: now also U1.D8; no longer U1.D4
- net PRESENCE_2: now also U1.D9; no longer U1.D7
- net PRESENCE_3: now also U1.D10; no longer U1.D8
- net PRESENCE_4: now also U1.D11; no longer U1.D10
- net PRESENCE_5: now also U1.D12; no longer U1.D11
Changed lines of the file:
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@@
 </signal>
 <signal name="N$39">
+<contactref element="R10" pad="P$2"/>
 <contactref element="U1" pad="D5"/>
-<contactref element="R10" pad="P$2"/>
 <wire x1="1032.7852375" y1="701.894146875" x2="1090.83673125" y2="657.0113" width="0" layer="19" extent="1-1"/>
-</signal>
-<signal name="N$40">
-<contactref element="U1" pad="D6"/>
-<contactref element="R9" pad="P$2"/>
-<wire x1="1036.6818125" y1="703.67811875" x2="1093.036434375" y2="655.7413" width="0" layer="19" extent="1-1"/>
 </signal>
 <signal name="N$41">
@@
 <signal name="N$45">
 <contactref element="R8" pad="P$2"/>
-<contactref element="U1" pad="D9"/>
-<wire x1="1025.64251875" y1="705.2957375" x2="1100.7354" y2="651.2963" width="0" layer="19" extent="1-1"/>
+<contactref element="U1" pad="D6"/>
+<wire x1="1025.64251875" y1="705.2957375" x2="1093.036434375" y2="655.7413" width="0" layer="19" extent="1-1"/>
 </signal>
 <signal name="N$46">
 <contactref element="IHM" pad="1"/>
-<contactref element="U1" pad="D3"/>
 <contactref element="R11" pad="P$1"/>
-<wire x1="1086.437321875" y1="659.5513" x2="1019.976734375" y2="701.23383125" width="0" layer="19" extent="1-1"/>
 <wire x1="1031.338584375" y1="720.126840625" x2="1019.976734375" y2="701.23383125" width="0.8128" layer="16"/>
+<contactref element="U1" pad="D7"/>
+<wire x1="1019.976734375" y1="701.23383125" x2="1095.236140625" y2="654.4713" width="0" layer="19" extent="1-1"/>
 </signal>
 <signal name="N$47">
 <contactref element="IHM" pad="4"/>
-<contactref element="U1" pad="D2"/>
 <contactref element="R12" pad="P$1"/>
-<wire x1="1084.237615625" y1="660.8213" x2="1032.272346875" y2="706.786896875" width="0" layer="19" extent="1-1"/>
 <wire x1="1037.9377" y1="716.316840625" x2="1032.272346875" y2="706.786896875" width="0.8128" layer="16"/>
+<contactref element="U1" pad="D4"/>
+<wire x1="1032.272346875" y1="706.786896875" x2="1088.637025" y2="658.2813" width="0" layer="19" extent="1-1"/>
 </signal>
 <signal name="PRESENCE_1">
-<contactref element="U1" pad="D4"/>
 <contactref element="R14" pad="P$1"/>
-<wire x1="986.35035" y1="666.610615625" x2="1088.637025" y2="658.2813" width="0" layer="19" extent="1-1"/>
+<contactref element="U1" pad="D8"/>
+<wire x1="986.35035" y1="666.610615625" x2="1098.535696875" y2="652.5663" width="0" layer="19" extent="1-1"/>
 </signal>
 <signal name="PRESENCE_2">
-<contactref element="U1" pad="D7"/>
 <contactref element="R15" pad="P$1"/>
-<wire x1="983.5022375" y1="668.03173125" x2="1095.236140625" y2="654.4713" width="0" layer="19" extent="1-1"/>
+<contactref element="U1" pad="D9"/>
+<wire x1="983.5022375" y1="668.03173125" x2="1100.7354" y2="651.2963" width="0" layer="19" extent="1-1"/>
 </signal>
 <signal name="PRESENCE_3">
-<contactref element="U1" pad="D8"/>
 <contactref element="R16" pad="P$1"/>
-<wire x1="980.45165" y1="669.65873125" x2="1098.535696875" y2="652.5663" width="0" layer="19" extent="1-1"/>
+<contactref element="U1" pad="D10"/>
+<wire x1="980.45165" y1="669.65873125" x2="1102.93510625" y2="650.0263" width="0" layer="19" extent="1-1"/>
 </signal>
 <signal name="PRESENCE_4">
-<contactref element="U1" pad="D10"/>
 <contactref element="R17" pad="P$1"/>
-<wire x1="977.53005" y1="671.40873125" x2="1102.93510625" y2="650.0263" width="0" layer="19" extent="1-1"/>
+<contactref element="U1" pad="D11"/>
+<wire x1="977.53005" y1="671.40873125" x2="1105.134809375" y2="648.7563" width="0" layer="19" extent="1-1"/>
 </signal>
 <signal name="PRESENCE_5">
-<contactref element="U1" pad="D11"/>
 <contactref element="R18" pad="P$1"/>
-<wire x1="973.526459375" y1="672.241734375" x2="1105.134809375" y2="648.7563" width="0" layer="19" extent="1-1"/>
+<contactref element="U1" pad="D12"/>
+<wire x1="973.526459375" y1="672.241734375" x2="1107.3345125" y2="647.4863" width="0" layer="19" extent="1-1"/>
 </signal>
 <signal name="N$49">
 <contactref element="IHM" pad="7"/>
 <contactref element="R13" pad="P$1"/>
-<contactref element="U1" pad="D12"/>
-<wire x1="1107.3345125" y1="647.4863" x2="1039.988421875" y2="702.6512625" width="0" layer="19" extent="1-1"/>
 <wire x1="1044.5368125" y1="712.50684375" x2="1039.988421875" y2="702.6512625" width="0.8128" layer="16"/>
+<contactref element="U1" pad="D2"/>
+<wire x1="1039.988421875" y1="702.6512625" x2="1084.237615625" y2="660.8213" width="0" layer="19" extent="1-1"/>
 </signal>
 <signal name="N$50">
@@
 <wire x1="1171.194" y1="833.374" x2="1171.194" y2="830.58" width="0.8128" layer="16"/>
 </signal>
+<signal name="N$17">
+<contactref element="R9" pad="P$2"/>
+<contactref element="U1" pad="D3"/>
+<wire x1="1036.6818125" y1="703.67811875" x2="1086.437321875" y2="659.5513" width="0" layer="19" extent="1-1"/>
+</signal>
 </signals>

Commit message: [AIIO_boards] Route presence connectors.
Parts:
- moved U$4 383.7 mm to (1229.8, 685.8), turned to 318 degrees
- moved BAT_12V_PROPU 353.2 mm to (1228.6, 712.3), turned to 61 degrees
- moved U$5 323.7 mm to (1268.5, 683.7), turned to 42 degrees
- moved 12V_PROPU_SRC 316.7 mm to (1235.4, 724.3), turned to 240 degrees
- moved R19 298.5 mm to (1243.0, 704.8), turned to 216 degrees
- moved LED4 288.5 mm to (1252.1, 710.4), turned to 126 degrees
- moved U$6 288.3 mm to (1259.2, 693.4), turned to 36 degrees
- moved 12V_PROPU_SRC1 281.7 mm to (1241.6, 735.2), turned to 240 degrees
- moved JP7 277.2 mm to (1171.2, 698.0), turned to 90 degrees
- moved JP6 267.9 mm to (1162.8, 698.0), turned to 90 degrees
- moved JP4 253.9 mm to (1145.3, 698.0), turned to 90 degrees
- moved JP5 253.3 mm to (1153.9, 698.0), turned to 90 degrees
- moved JP3 240.8 mm to (1136.7, 698.0), turned to 90 degrees
- moved R18 145.1 mm to (1120.0, 663.5), turned to 150 degrees
- moved R17 136.8 mm to (1115.7, 663.5), turned to 150 degrees
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Connections:
- net GND: now also JP3.2, JP4.2, JP5.2, JP6.2, JP7.2; no longer JP6.1
- net PRESENCE_1: now also JP3.1
- net PRESENCE_2: now also JP4.1
- net PRESENCE_3: now also JP5.1
- net PRESENCE_4: now also JP6.1
- net PRESENCE_5: now also JP7.1
Routing:
- net N$46: track 22.0 -> 148.0 mm
- net N$45: track 0.00 -> 125.0 mm
- net N$47: track 11.1 -> 126.4 mm
- net N$39: track 0.00 -> 114.4 mm
- net N$17: track 0.00 -> 107.1 mm
- net N$49: track 10.9 -> 108.9 mm
- net TX_RP2: track 0.00 -> 95.7 mm
- net RX_RP2: track 0.00 -> 94.0 mm
- net PRESENCE_5: track 0.00 -> 86.7 mm
- net PRESENCE_4: track 0.00 -> 80.2 mm
- net PRESENCE_3: track 0.00 -> 73.4 mm
- net PRESENCE_2: track 0.00 -> 68.3 mm
- net PRESENCE_1: track 0.00 -> 67.0 mm
- net SCL_ARDU: track 0.00 -> 61.8 mm
- net SDA_ARDU: track 0.00 -> 56.3 mm
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