File: 2017/primary/primary_teensy.sch (EAGLE design)
At the start: 46 parts, among them IC1 74LS241N, Q1 MFR475V, Q2 MFR475V

Commit message: [Primary] Erase some componants.
Parts:
- removed JP1: (no value), pinhead:PINHD-1X8
- removed RP1: RASPI_BOARD_B+#_FP, raspberrypi_bastelstube_v13-enac:RASPI_BOARD_B+#_FP
Connections:
- removed net 5V_RPI: JP1.1, RP1.5V0A
- removed net GND_RPI: JP1.2, RP1.GND_A
- removed net RP2_PWR: JP1.8, RP1.SPI_CE1
- removed net RPI_04: JP1.7, RP1.GPIO04
- removed net RX_RPI: JP1.4, RP1.RXD
- removed net SCL_RPI: JP1.6, RP1.SCL
- removed net SDA_RPI: JP1.5, RP1.SDA
- removed net TX_RPI: JP1.3, RP1.TXD
- net GND: now also U$1.GND
Changed lines of the file:
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@@
 </part>
 <part name="JUMPER_ALIM" library="pinhead" deviceset="PINHD-1X2" device=""/>
-<part name="JP1" library="pinhead" deviceset="PINHD-1X8" device=""/>
 <part name="C7" library="resistor" deviceset="CPOL-EU" device="E5-13" value="2.2m"/>
 <part name="C8" library="resistor" deviceset="CPOL-EU" device="E5-13" value="2.2m"/>
@@
 <attribute name="OC_NEWARK" value="unknown"/>
 </part>
-<part name="RP1" library="raspberrypi_bastelstube_v13-enac" deviceset="RASPI_BOARD_B+#" device="_FP"/>
 </parts>
 <sheets>
@@
 <instance part="5V_PWR" gate="-2" x="170.18" y="58.42"/>
 <instance part="JUMPER_ALIM" gate="G$1" x="27.94" y="12.7"/>
-<instance part="JP1" gate="A" x="325.12" y="17.78" rot="R90"/>
 <instance part="C7" gate="G$1" x="-25.4" y="96.52" rot="R180"/>
 <instance part="C8" gate="G$1" x="33.02" y="96.52" rot="R270"/>
@@
 <instance part="12V_PWR_BOARD1" gate="-1" x="114.3" y="99.06"/>
 <instance part="12V_PWR_BOARD1" gate="-2" x="114.3" y="93.98"/>
-<instance part="RP1" gate="G$1" x="322.58" y="-45.72"/>
 </instances>
 <busses>
@@
 <label x="180.34" y="58.42" size="1.778" layer="95"/>
 </segment>
+<segment>
+<pinref part="U$1" gate="G$1" pin="GND"/>
+<wire x1="-20.32" y1="12.7" x2="-30.48" y2="12.7" width="0.1524" layer="91"/>
+<label x="-30.48" y="12.7" size="1.778" layer="95"/>
+</segment>
 </net>
 <net name="N$4" class="0">
@@
 <pinref part="R3" gate="G$1" pin="2"/>
 <pinref part="U$3" gate="G$1" pin="TRM"/>
-</segment>
-</net>
-<net name="TX_RPI" class="0">
-<segment>
-<wire x1="337.82" y1="-45.72" x2="350.52" y2="-45.72" width="0.1524" layer="91"/>
-<wire x1="350.52" y1="-45.72" x2="350.52" y2="-2.54" width="0.1524" layer="91"/>
-<pinref part="JP1" gate="A" pin="3"/>
-<wire x1="350.52" y1="-2.54" x2="320.04" y2="-2.54" width="0.1524" layer="91"/>
-<wire x1="320.04" y1="-2.54" x2="320.04" y2="15.24" width="0.1524" layer="91"/>
-<pinref part="RP1" gate="G$1" pin="TXD"/>
-</segment>
-</net>
-<net name="RX_RPI" class="0">
-<segment>
-<wire x1="337.82" y1="-48.26" x2="353.06" y2="-48.26" width="0.1524" layer="91"/>
-<wire x1="353.06" y1="-48.26" x2="353.06" y2="0" width="0.1524" layer="91"/>
-<pinref part="JP1" gate="A" pin="4"/>
-<wire x1="353.06" y1="0" x2="322.58" y2="0" width="0.1524" layer="91"/>
-<wire x1="322.58" y1="0" x2="322.58" y2="15.24" width="0.1524" layer="91"/>
-<pinref part="RP1" gate="G$1" pin="RXD"/>
-</segment>
-</net>
-<net name="RPI_04" class="0">
-<segment>
-<wire x1="307.34" y1="-48.26" x2="304.8" y2="-48.26" width="0.1524" layer="91"/>
-<wire x1="304.8" y1="-48.26" x2="304.8" y2="5.08" width="0.1524" layer="91"/>
-<pinref part="JP1" gate="A" pin="7"/>
-<wire x1="304.8" y1="5.08" x2="330.2" y2="5.08" width="0.1524" layer="91"/>
-<wire x1="330.2" y1="5.08" x2="330.2" y2="15.24" width="0.1524" layer="91"/>
-<pinref part="RP1" gate="G$1" pin="GPIO04"/>
-</segment>
-</net>
-<net name="RP2_PWR" class="0">
-<segment>
-<wire x1="337.82" y1="-40.64" x2="345.44" y2="-40.64" width="0.1524" layer="91"/>
-<wire x1="345.44" y1="-40.64" x2="345.44" y2="7.62" width="0.1524" layer="91"/>
-<pinref part="JP1" gate="A" pin="8"/>
-<wire x1="345.44" y1="7.62" x2="332.74" y2="7.62" width="0.1524" layer="91"/>
-<wire x1="332.74" y1="7.62" x2="332.74" y2="15.24" width="0.1524" layer="91"/>
-<pinref part="RP1" gate="G$1" pin="SPI_CE1"/>
-</segment>
-</net>
-<net name="SCL_RPI" class="0">
-<segment>
-<wire x1="302.26" y1="-78.74" x2="307.34" y2="-78.74" width="0.1524" layer="91"/>
-<wire x1="302.26" y1="-78.74" x2="302.26" y2="7.62" width="0.1524" layer="91"/>
-<wire x1="302.26" y1="7.62" x2="327.66" y2="7.62" width="0.1524" layer="91"/>
-<pinref part="JP1" gate="A" pin="6"/>
-<wire x1="327.66" y1="7.62" x2="327.66" y2="15.24" width="0.1524" layer="91"/>
-<pinref part="RP1" gate="G$1" pin="SCL"/>
-</segment>
-</net>
-<net name="SDA_RPI" class="0">
-<segment>
-<wire x1="307.34" y1="-81.28" x2="299.72" y2="-81.28" width="0.1524" layer="91"/>
-<wire x1="299.72" y1="-81.28" x2="299.72" y2="10.16" width="0.1524" layer="91"/>
-<pinref part="JP1" gate="A" pin="5"/>
-<wire x1="299.72" y1="10.16" x2="325.12" y2="10.16" width="0.1524" layer="91"/>
-<wire x1="325.12" y1="10.16" x2="325.12" y2="15.24" width="0.1524" layer="91"/>
-<pinref part="RP1" gate="G$1" pin="SDA"/>
 </segment>
 </net>
@@
 </segment>
 </net>
-<net name="5V_RPI" class="0">
-<segment>
-<wire x1="314.96" y1="-17.78" x2="314.96" y2="15.24" width="0.1524" layer="91"/>
-<pinref part="JP1" gate="A" pin="1"/>
-<pinref part="RP1" gate="G$1" pin="5V0A"/>
-</segment>
-</net>
-<net name="GND_RPI" class="0">
-<segment>
-<wire x1="355.6" y1="-53.34" x2="337.82" y2="-53.34" width="0.1524" layer="91"/>
-<wire x1="355.6" y1="-53.34" x2="355.6" y2="2.54" width="0.1524" layer="91"/>
-<pinref part="JP1" gate="A" pin="2"/>
-<wire x1="355.6" y1="2.54" x2="317.5" y2="2.54" width="0.1524" layer="91"/>
-<wire x1="317.5" y1="2.54" x2="317.5" y2="15.24" width="0.1524" layer="91"/>
-<pinref part="RP1" gate="G$1" pin="GND_A"/>
-</segment>
-</net>

Commit message: [primary] 2nd version, without mass plane.
Parts:
- removed LED: (no value), pinhead:PINHD-1X2
- added LED_RGB: (no value), pinhead:PINHD-1X4
- added R4, R5, R6: (no value), resistor:R-EU_0207/7
Connections:
- new net N$11: LED_RGB.2, R4.1
- new net N$19: R6.2, U$1.36/A17
- new net N$20: IHM_BONUS.2, U$1.35/A16
- new net N$3: LED_RGB.4, R6.1
- new net N$7: LED_RGB.3, R5.1
- net 5V_SIG: now also IC1P.VCC
- net GND: now also IC1P.GND, LED_RGB.1; no longer LED.1
- net MOT_LANCEUR: now also U$1.30; no longer U$1.35/A16
- net MOT_RAMASSAGE: now also U$1.29; no longer U$1.36/A17
- net N$17: now also R4.2, U$1.38/A19; no longer LED.2, U$1.29
- net N$18: now also R5.2, U$1.37/A18; no longer IHM_BONUS.2, U$1.30
Other:
- moved on the sheet: D1, D2, IHM_BONUS, JUMPER_MOTEUR_LANCEUR, JUMPER_MOTEUR_RAMASSAGE, MOTEUR_LANCEUR-1, MOTEUR_LANCEUR-2, MOTEUR_RAMASSAGE-1, MOTEUR_RAMASSAGE-2, Q1, Q2, R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
