File: 2017/primary/primary_teensy.brd (EAGLE design)
At the start: 46 parts, among them IC1 74LS241N, Q1 MFR475V, Q2 MFR475V

Commit message: [Primary] Erase some componants.
Parts:
- removed JP1: (no value), pinhead:1X08
- removed RP1: RASPI_BOARD_B+#_FP, raspberrypi_bastelstube_v13-enac:RASPI_BOARD_B+_FULL_PAD
Connections:
- removed net 3V3A: RP1.1
- removed net 3V3B: RP1.17
- removed net 5V0B: RP1.4
- removed net 5V_RPI: JP1.1, RP1.2
- removed net GND_B: RP1.9
- removed net GND_C: RP1.14
- removed net GND_D: RP1.20
- removed net GND_E: RP1.25
- removed net GND_F: RP1.30
- removed net GND_G: RP1.34
- removed net GND_H: RP1.39
- removed net GND_RPI: JP1.2, RP1.6
- removed net RP2_PWR: JP1.8, RP1.26
- removed net RPI_04: JP1.7, RP1.7
- removed net RX_RPI: JP1.4, RP1.10
- removed net SCL_RPI: JP1.6, RP1.5
- removed net SDA_RPI: JP1.5, RP1.3
- removed net TX_RPI: JP1.3, RP1.8
- net GND: now also U$1.GND
Routing:
- net GND: track 497.6 -> 520.1 mm
- net 5V_SIG: track 224.3 -> 225.4 mm
Changed lines of the file:
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@@
 </element>
 <element name="JUMPER_ALIM" library="pinhead" package="1X02" value="" x="1089.678" y="537.2094" rot="R270"/>
-<element name="JP1" library="pinhead" package="1X08" value="" x="1263.675" y="502.78"/>
 <element name="C7" library="resistor" package="E5-13" value="2.2m" x="970.28" y="523.24"/>
 <element name="C8" library="resistor" package="E5-13" value="2.2m" x="1031.24" y="477.52" rot="R180"/>
@@
 <attribute name="OC_FARNELL" value="unknown" x="1140.46" y="533.4" size="1.778" layer="27" rot="R180" display="off"/>
 </element>
-<element name="RP1" library="raspberrypi_bastelstube_v13-enac" package="RASPI_BOARD_B+_FULL_PAD" value="RASPI_BOARD_B+#_FP" x="1233.805" y="476.885"/>
 </elements>
 <signals>
@@
 <wire x1="1089.66" y1="472.44" x2="1089.66" y2="464.82" width="1.27" layer="16"/>
 <wire x1="1089.66" y1="464.82" x2="1089.66" y2="459.74" width="1.27" layer="16"/>
+<contactref element="U$1" pad="GND"/>
 <wire x1="1112.5128" y1="533.4072" x2="1112.5266" y2="533.4066" width="0" layer="19" extent="16-16"/>
 <wire x1="1099.829" y1="474.98" x2="1099.82" y2="474.98" width="0" layer="19" extent="16-16"/>
@@
 <wire x1="1051.5464" y1="482.6076" x2="1051.5464" y2="482.5864" width="0" layer="19" extent="16-16"/>
 <wire x1="1130.3" y1="518.16" x2="1130.2788" y2="518.1826" width="0" layer="19" extent="16-16"/>
+<wire x1="1066.777" y1="535.906" x2="1066.777" y2="535.963" width="1.016" layer="16"/>
+<wire x1="1066.777" y1="535.963" x2="1062.99" y2="539.75" width="1.016" layer="16"/>
+<wire x1="1062.99" y1="539.75" x2="1050.29" y2="539.75" width="1.016" layer="16"/>
+<wire x1="1050.29" y1="539.75" x2="1049.02" y2="538.48" width="1.016" layer="16"/>
+<wire x1="1049.02" y1="538.48" x2="1049.02" y2="535.936" width="1.016" layer="16"/>
+<wire x1="1049.02" y1="535.936" x2="1049.0252" y2="535.9308" width="1.016" layer="16"/>
 </signal>
 <signal name="N$4">
@@
 <wire x1="1016" y1="467.36" x2="1016" y2="474.98" width="1.27" layer="16"/>
 </signal>
-<signal name="3V3A">
-<contactref element="RP1" pad="1"/>
-</signal>
-<signal name="5V0B">
-<contactref element="RP1" pad="4"/>
-</signal>
-<signal name="3V3B">
-<contactref element="RP1" pad="17"/>
-</signal>
-<signal name="GND_B">
-<contactref element="RP1" pad="9"/>
-</signal>
-<signal name="GND_C">
-<contactref element="RP1" pad="14"/>
-</signal>
-<signal name="GND_D">
-<contactref element="RP1" pad="20"/>
-</signal>
-<signal name="GND_E">
-<contactref element="RP1" pad="25"/>
-</signal>
-<signal name="GND_F">
-<contactref element="RP1" pad="30"/>
-</signal>
-<signal name="GND_G">
-<contactref element="RP1" pad="34"/>
-</signal>
-<signal name="GND_H">
-<contactref element="RP1" pad="39"/>
-</signal>
-<signal name="TX_RPI">
-<contactref element="JP1" pad="3"/>
-<contactref element="RP1" pad="8"/>
-<wire x1="1259.865" y1="502.78" x2="1249.795" y2="530.655" width="0" layer="19" extent="1-1"/>
-</signal>
-<signal name="RX_RPI">
-<contactref element="JP1" pad="4"/>
-<contactref element="RP1" pad="10"/>
-<wire x1="1262.405" y1="502.78" x2="1252.335" y2="530.655" width="0" layer="19" extent="1-1"/>
-</signal>
-<signal name="RPI_04">
-<contactref element="JP1" pad="7"/>
-<contactref element="RP1" pad="7"/>
-<wire x1="1249.795" y1="528.115" x2="1270.025" y2="502.78" width="0" layer="19" extent="1-1"/>
-</signal>
 <signal name="N$50">
-</signal>
-<signal name="RP2_PWR">
-<contactref element="JP1" pad="8"/>
-<contactref element="RP1" pad="26"/>
-<wire x1="1272.565" y1="502.78" x2="1272.655" y2="530.655" width="0" layer="19" extent="1-1"/>
-</signal>
-<signal name="SCL_RPI">
-<contactref element="JP1" pad="6"/>
-<contactref element="RP1" pad="5"/>
-<wire x1="1247.255" y1="528.115" x2="1267.485" y2="502.78" width="0" layer="19" extent="1-1"/>
-</signal>
-<signal name="SDA_RPI">
-<contactref element="JP1" pad="5"/>
-<contactref element="RP1" pad="3"/>
-<wire x1="1244.715" y1="528.115" x2="1264.945" y2="502.78" width="0" layer="19" extent="1-1"/>
 </signal>
 <signal name="5V_SIG">
@@
 <wire x1="1046.48" y1="535.9256" x2="1046.4852" y2="535.9308" width="1.016" layer="16"/>
 <wire x1="1046.4852" y1="535.9308" x2="1046.4852" y2="538.4852" width="1.016" layer="16"/>
-<wire x1="1046.4852" y1="538.4852" x2="1049.02" y2="541.02" width="1.016" layer="16"/>
-<wire x1="1049.02" y1="541.02" x2="1087.12" y2="541.02" width="1.016" layer="16"/>
+<wire x1="1046.4852" y1="538.4852" x2="1050.29" y2="542.29" width="1.016" layer="16"/>
+<wire x1="1050.29" y1="542.29" x2="1064.26" y2="542.29" width="1.016" layer="16"/>
+<wire x1="1064.26" y1="542.29" x2="1065.53" y2="541.02" width="1.016" layer="16"/>
+<wire x1="1065.53" y1="541.02" x2="1087.12" y2="541.02" width="1.016" layer="16"/>
 <wire x1="1102.3748" y1="495.3052" x2="1094.769" y2="495.3052" width="1.016" layer="16"/>
 <wire x1="1094.769" y1="495.3052" x2="1094.7452" y2="495.3052" width="1.016" layer="16"/>
@@
 <wire x1="1082.0504" y1="535.9394" x2="1082.017" y2="535.906" width="1.016" layer="16"/>
 </signal>
-<signal name="5V_RPI">
-<contactref element="JP1" pad="1"/>
-<contactref element="RP1" pad="2"/>
-<wire x1="1254.785" y1="502.78" x2="1242.175" y2="530.655" width="0" layer="19" extent="1-1"/>
-</signal>
-<signal name="GND_RPI">
-<contactref element="JP1" pad="2"/>
-<contactref element="RP1" pad="6"/>
-<wire x1="1257.325" y1="502.78" x2="1247.255" y2="530.655" width="0" layer="19" extent="1-1"/>
-</signal>
 </signals>

Commit message: [primary] 2nd version, without mass plane.
Parts:
- removed LED: (no value), pinhead:1X02
- added LED_RGB: (no value), pinhead:1X04
- added R4, R5, R6: (no value), resistor:0207/7
- moved C7 204.7 mm to (1170.9, 482.6), turned to 180 degrees
- moved 3V3_PWR1 153.2 mm to (1003.3, 518.2), turned to 270 degrees
- moved U$3 151.9 mm to (1144.3, 478.8), turned to 90 degrees
- moved 12V_BOARD1 148.6 mm to (1154.4, 535.9)
- moved MOTEUR_LANCEUR 140.3 mm to (1003.3, 482.6), turned to 270 degrees
- moved 12V_PWR_BOARD1 140.0 mm to (1003.3, 505.5), turned to 270 degrees
- moved MOTEUR_RAMASSAGE 139.8 mm to (1003.3, 492.7), turned to 270 degrees
- moved R3 137.9 mm to (1130.3, 534.7), turned to 180 degrees
- moved R2 134.1 mm to (1130.3, 530.9), turned to 180 degrees
- moved REGU_3V1 120.9 mm to (1017.3, 518.2)
- moved C4 118.2 mm to (1014.7, 508.0), turned to 270 degrees
- moved C5 115.8 mm to (1017.3, 525.8), turned to 0 degrees
- moved D1 104.4 mm to (1018.5, 480.1), turned to 0 degrees
- moved D2 104.2 mm to (1018.5, 490.2), turned to 0 degrees
- moved C8 91.4 mm to (1112.5, 519.4), turned to 0 degrees
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Connections:
- removed net VCC: IC1.20
- new net N$11: LED_RGB.2, R4.1
- new net N$19: R6.2, U$1.36/A17
- new net N$20: IHM_BONUS.2, U$1.35/A16
- new net N$3: LED_RGB.4, R6.1
- new net N$7: LED_RGB.3, R5.1
- net 5V_SIG: now also IC1.20
- net GND: now also LED_RGB.1; no longer LED.1
- net MOT_LANCEUR: now also U$1.30; no longer U$1.35/A16
- net MOT_RAMASSAGE: now also U$1.29; no longer U$1.36/A17
- net N$17: now also R4.2, U$1.38/A19; no longer LED.2, U$1.29
- net N$18: now also R5.2, U$1.37/A18; no longer IHM_BONUS.2, U$1.30
Routing:
- net GND: track 520.1 -> 0.00 mm, vias 2 -> 0
- net 12V_PWR: track 168.1 -> 113.5 mm
- net GND_12: track 44.4 -> 96.1 mm
- net 3V3: track 60.5 -> 16.5 mm, vias 2 -> 0
- net TX4: track 10.1 -> 43.9 mm
- net N$45: track 40.2 -> 8.89 mm
- net +12V: track 63.7 -> 92.7 mm
- net RX4: track 14.5 -> 41.0 mm
- net N$20: track 0.00 -> 18.8 mm
- net N$10: track 27.5 -> 12.0 mm
- net N$13: track 27.5 -> 14.1 mm
- net N$14: track 29.6 -> 16.4 mm
- net N$12: track 25.4 -> 12.5 mm
- net N$18: track 14.8 -> 5.12 mm
- net N$17: track 13.8 -> 5.12 mm
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
Commit message: [primary] Adds mass plane.
Routing:
- net GND: track 0.00 -> 96.6 mm, vias 0 -> 10
- added copper zone on layer 16, net GND
Changed lines of the file:
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@@
 <param name="mtCopper" value="0.035mm 0.035mm 0.035mm 0.035mm 0.035mm 0.035mm 0.035mm 0.035mm 0.035mm 0.035mm 0.035mm 0.035mm 0.035mm 0.035mm 0.035mm 0.035mm"/>
 <param name="mtIsolate" value="1.5mm 0.15mm 0.2mm 0.15mm 0.2mm 0.15mm 0.2mm 0.15mm 0.2mm 0.15mm 0.2mm 0.15mm 0.2mm 0.15mm 0.2mm"/>
-<param name="mdWireWire" value="15mil"/>
-<param name="mdWirePad" value="15mil"/>
-<param name="mdWireVia" value="15mil"/>
+<param name="mdWireWire" value="30mil"/>
+<param name="mdWirePad" value="30mil"/>
+<param name="mdWireVia" value="30mil"/>
 <param name="mdPadPad" value="15mil"/>
 <param name="mdPadVia" value="15mil"/>
@@
 <contactref element="IHM_BONUS" pad="1"/>
 <contactref element="IC1" pad="10"/>
-<wire x1="1014.73" y1="518.16" x2="1003.3" y2="520.6746" width="0" layer="19" extent="1-1"/>
-<wire x1="1019.8312" y1="525.7574" x2="1014.73" y2="518.16" width="0" layer="19" extent="1-1"/>
-<wire x1="1014.73" y1="505.46" x2="1014.73" y2="518.16" width="0" layer="19" extent="1-1"/>
-<wire x1="1023.6224" y1="506.7462" x2="1014.73" y2="505.46" width="0" layer="19" extent="1-1"/>
-<wire x1="1003.3" y1="502.9708" x2="1014.73" y2="505.46" width="0" layer="19" extent="1-1"/>
-<wire x1="1031.24" y1="519.43" x2="1019.8312" y2="525.7574" width="0" layer="19" extent="1-1"/>
-<wire x1="1038.8652" y1="524.4986" x2="1031.24" y2="519.43" width="0" layer="19" extent="1-1"/>
-<wire x1="1046.4932" y1="519.4342" x2="1038.8652" y2="524.4986" width="0" layer="19" extent="1-1"/>
-<wire x1="1052.83" y1="524.51" x2="1046.4932" y2="519.4342" width="0" layer="19" extent="1-1"/>
-<wire x1="1052.8248" y1="532.1508" x2="1052.83" y2="524.51" width="0" layer="19" extent="1-1"/>
-<wire x1="1052.8352" y1="541.0108" x2="1052.8248" y2="532.1508" width="0" layer="19" extent="1-1"/>
-<wire x1="1038.8558" y1="513.0968" x2="1031.24" y2="519.43" width="0" layer="19" extent="1-1"/>
-<wire x1="1055.3796" y1="514.3458" x2="1046.4932" y2="519.4342" width="0" layer="19" extent="1-1"/>
-<wire x1="1055.309" y1="504.135" x2="1055.3796" y2="514.3458" width="0" layer="19" extent="1-1"/>
-<wire x1="1055.3564" y1="497.8334" x2="1055.309" y2="504.135" width="0" layer="19" extent="1-1"/>
-<wire x1="1055.3564" y1="492.7478" x2="1055.3564" y2="497.8334" width="0" layer="19" extent="1-1"/>
-<wire x1="1066.777" y1="535.906" x2="1052.8248" y2="532.1508" width="0" layer="19" extent="1-1"/>
-<wire x1="1029.9668" y1="492.7398" x2="1023.6224" y2="506.7462" width="0" layer="19" extent="1-1"/>
-<wire x1="1033.8002" y1="477.5148" x2="1029.9668" y2="492.7398" width="0" layer="19" extent="1-1"/>
-<wire x1="1098.5428" y1="529.5972" x2="1066.777" y2="535.906" width="0" layer="19" extent="1-1"/>
-<wire x1="1098.5428" y1="523.2416" x2="1098.5428" y2="529.5972" width="0" layer="19" extent="1-1"/>
-<wire x1="1098.5428" y1="516.886" x2="1098.5428" y2="523.2416" width="0" layer="19" extent="1-1"/>
-<wire x1="1098.5458" y1="510.5576" x2="1098.5428" y2="516.886" width="0" layer="19" extent="1-1"/>
-<wire x1="1106.2268" y1="535.9466" x2="1098.5428" y2="529.5972" width="0" layer="19" extent="1-1"/>
-<wire x1="1099.8348" y1="500.3852" x2="1098.5458" y2="510.5576" width="0" layer="19" extent="1-1"/>
-<wire x1="1092.229" y1="500.3852" x2="1099.8348" y2="500.3852" width="0" layer="19" extent="1-1"/>
-<wire x1="1099.82" y1="492.76" x2="1099.8348" y2="500.3852" width="0" layer="19" extent="1-1"/>
-<wire x1="1099.818" y1="477.5064" x2="1099.82" y2="492.76" width="0" layer="19" extent="1-1"/>
-<wire x1="1115.06" y1="519.43" x2="1098.5428" y2="516.886" width="0" layer="19" extent="1-1"/>
-<wire x1="1136.65" y1="524.51" x2="1115.06" y2="519.43" width="0" layer="19" extent="1-1"/>
-<wire x1="1134.11" y1="530.86" x2="1136.65" y2="524.51" width="0" layer="19" extent="1-1"/>
+<polygon width="1.016" layer="16">
+<vertex x="1181.1" y="473.71"/>
+<vertex x="995.68" y="473.71"/>
+<vertex x="995.68" y="529.59"/>
+<vertex x="1045.21" y="529.59"/>
+<vertex x="1045.21" y="547.37"/>
+<vertex x="1162.05" y="547.37"/>
+<vertex x="1162.05" y="530.86"/>
+<vertex x="1178.56" y="530.86"/>
+<vertex x="1181.1" y="530.86"/>
+</polygon>
+<wire x1="1055.309" y1="504.135" x2="1060.395" y2="504.135" width="1.016" layer="16"/>
+<wire x1="1060.395" y1="504.135" x2="1060.45" y2="504.19" width="1.016" layer="16"/>
+<via x="1060.45" y="504.19" extent="1-16" drill="0.6" shape="square"/>
+<wire x1="1060.45" y1="504.19" x2="1060.45" y2="511.81" width="1.016" layer="1"/>
+<via x="1060.45" y="511.81" extent="1-16" drill="0.6" shape="square"/>
+<wire x1="1060.45" y1="511.81" x2="1057.91" y2="514.35" width="1.016" layer="16"/>
+<wire x1="1057.91" y1="514.35" x2="1055.3838" y2="514.35" width="1.016" layer="16"/>
+<wire x1="1055.3838" y1="514.35" x2="1055.3796" y2="514.3458" width="1.016" layer="16"/>
+<wire x1="1046.4932" y1="519.4342" x2="1043.9442" y2="519.4342" width="1.016" layer="16"/>
+<wire x1="1043.9442" y1="519.4342" x2="1043.94" y2="519.43" width="1.016" layer="16"/>
+<via x="1043.94" y="519.43" extent="1-16" drill="0.6" shape="square"/>
+<wire x1="1043.94" y1="519.43" x2="1038.86" y2="519.43" width="1.016" layer="1"/>
+<via x="1038.86" y="519.43" extent="1-16" drill="0.6" shape="square"/>
+<wire x1="1038.86" y1="519.43" x2="1038.86" y2="524.4934" width="1.016" layer="16"/>
+<wire x1="1038.86" y1="524.4934" x2="1038.8652" y2="524.4986" width="1.016" layer="16"/>
+<wire x1="1046.4932" y1="519.4342" x2="1046.4932" y2="513.0668" width="1.016" layer="16"/>
+<wire x1="1046.4932" y1="513.0668" x2="1047.75" y2="511.81" width="1.016" layer="16"/>
+<via x="1047.75" y="511.81" extent="1-16" drill="0.6" shape="square"/>
+<wire x1="1047.75" y1="511.81" x2="1052.83" y2="511.81" width="1.016" layer="1"/>
+<via x="1052.83" y="511.81" extent="1-16" drill="0.6" shape="square"/>
+<wire x1="1052.83" y1="511.81" x2="1054.1" y2="511.81" width="1.016" layer="16"/>
+<wire x1="1054.1" y1="511.81" x2="1055.37" y2="513.08" width="1.016" layer="16"/>
+<wire x1="1055.37" y1="513.08" x2="1055.37" y2="514.3362" width="1.016" layer="16"/>
+<wire x1="1055.37" y1="514.3362" x2="1055.3796" y2="514.3458" width="1.016" layer="16"/>
+<wire x1="1098.5458" y1="510.5576" x2="1103.6476" y2="510.5576" width="1.016" layer="16"/>
+<wire x1="1103.6476" y1="510.5576" x2="1107.44" y2="513.08" width="1.016" layer="16"/>
+<via x="1107.44" y="513.08" extent="1-16" drill="0.6" shape="square"/>
+<wire x1="1107.44" y1="513.08" x2="1112.52" y2="513.08" width="1.016" layer="1"/>
+<via x="1112.52" y="513.08" extent="1-16" drill="0.6" shape="square"/>
+<wire x1="1112.52" y1="513.08" x2="1115.06" y2="514.35" width="1.016" layer="16"/>
+<wire x1="1115.06" y1="514.35" x2="1118.87" y2="510.54" width="1.016" layer="16"/>
+<wire x1="1052.8248" y1="532.1508" x2="1052.83" y2="537.21" width="1.016" layer="16"/>
+<via x="1052.83" y="537.21" extent="1-16" drill="0.6" shape="square"/>
+<wire x1="1052.83" y1="537.21" x2="1061.72" y2="537.21" width="1.016" layer="1"/>
+<wire x1="1061.72" y1="537.21" x2="1064.26" y2="541.02" width="1.016" layer="1"/>
+<via x="1064.26" y="541.02" extent="1-16" drill="0.6" shape="square"/>
+<wire x1="1064.26" y1="541.02" x2="1066.8" y2="537.21" width="1.016" layer="16"/>
+<wire x1="1066.8" y1="537.21" x2="1066.777" y2="535.906" width="1.016" layer="16"/>
 </signal>
 <signal name="N$4">
@@
 <contactref element="R3" pad="1"/>
 <contactref element="IC1" pad="20"/>
-<wire x1="1050.29" y1="524.51" x2="1050.29" y2="541.02" width="1.016" layer="16"/>
 <wire x1="1050.29" y1="524.51" x2="1050.29" y2="502.92" width="1.016" layer="16"/>
 <wire x1="1050.29" y1="502.92" x2="1050.2762" y2="502.92" width="1.016" layer="16"/>
@@
 <wire x1="1093.47" y1="538.48" x2="1093.47" y2="535.9226" width="1.016" layer="16"/>
 <wire x1="1093.47" y1="535.9226" x2="1093.4694" y2="535.922" width="1.016" layer="16"/>
-<wire x1="1050.29" y1="541.02" x2="1050.2952" y2="541.0108" width="0" layer="19" extent="16-16"/>
-<wire x1="1050.2848" y1="532.1508" x2="1050.29" y2="524.51" width="0" layer="19" extent="1-1"/>
+<wire x1="1050.29" y1="524.51" x2="1050.2848" y2="532.1508" width="1.016" layer="16"/>
+<wire x1="1050.2848" y1="532.1508" x2="1050.2952" y2="541.0108" width="1.016" layer="16"/>
 </signal>
 <signal name="3V3">
@@
 <wire x1="1096.0028" y1="529.5972" x2="1096.0028" y2="523.2472" width="1.016" layer="16"/>
 <wire x1="1096.0028" y1="523.2472" x2="1096.01" y2="523.24" width="1.016" layer="16"/>
-<wire x1="1096.0028" y1="523.2472" x2="1096.0028" y2="523.2416" width="0" layer="19" extent="16-16"/>
 <wire x1="1096.0058" y1="510.5576" x2="1096.0058" y2="516.883" width="1.016" layer="16"/>
 <wire x1="1096.0058" y1="516.883" x2="1096.0028" y2="516.886" width="1.016" layer="16"/>
 <wire x1="1096.0028" y1="516.886" x2="1096.0028" y2="523.2416" width="1.016" layer="16"/>
+<wire x1="1096.0028" y1="523.2416" x2="1096.0028" y2="523.2472" width="0" layer="19" extent="16-16"/>
 </signal>
 <signal name="MOT_RAMASSAGE">
