File: 2018/jevois_pi/jevois_pi.sch (EAGLE design)
At the start: 8 parts, among them IC1 MAX3491ECSD+, IC2 MAX3491ECSD+, J1 TM21R-5C-88(50), J2 TM21R-5C-88(50), T1 R-78E3.3-0.5

Commit message: Correcting a mismatch between input pins
Connections:
- net RX1: now also JP1.3; no longer JP2.2
- net TX2: now also JP2.2; no longer JP1.3
Changed lines of the file:
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@@
 </segment>
 <segment>
-<pinref part="JP2" gate="A" pin="2"/>
-<wire x1="15.24" y1="86.36" x2="5.08" y2="86.36" width="0.1524" layer="91"/>
-<label x="5.08" y="86.36" size="1.778" layer="95"/>
+<pinref part="JP1" gate="A" pin="3"/>
+<wire x1="15.24" y1="106.68" x2="5.08" y2="106.68" width="0.1524" layer="91"/>
+<label x="5.08" y="106.68" size="1.778" layer="95"/>
 </segment>
 </net>
@@
 </segment>
 <segment>
-<pinref part="JP1" gate="A" pin="3"/>
-<wire x1="15.24" y1="106.68" x2="5.08" y2="106.68" width="0.1524" layer="91"/>
-<label x="5.08" y="106.68" size="1.778" layer="95"/>
+<pinref part="JP2" gate="A" pin="2"/>
+<wire x1="15.24" y1="86.36" x2="5.08" y2="86.36" width="0.1524" layer="91"/>
+<label x="5.08" y="86.36" size="1.778" layer="95"/>
 </segment>
 </net>
