File: 2018/secondary/secondary_18.sch (EAGLE design)
At the start: 9 parts

Commit message: [Secondary] Finishes the 2018 schematic
Parts:
- removed SV2: (no value), con-lstb:MA03-1
- added CON_I2C2_1, CON_I2C2_2, CON_I2C2_3, CON_I2C2_4, CON_I2C2_5, ENCOD1, SV3, UART: (no value), con-lstb:MA04-1
- added CON_MOT1, CON_MOT2, CON_SERV1, CON_SERV2, CON_SERV3: (no value), con-lstb:MA03-1
- added COULEUR, TIRETTE: (no value), pinhead:PINHD-1X2
- added D2, D3: 1N4004, diode:1N4004
- added DYNAMIX: (no value), con-lstb:MA05-1
- added Q1, Q2: BUZ11, transistor-fet:BUZ11
- added R2, R4: 10k, resistor:R-EU_0204/7
- added R3, R5: 10, resistor:R-EU_0204/7
- added SL1, SL2: (no value), con-amp-quick:MA02
- added U$3: DC-DC-STEP-DOWN-LM2596, diy-modules:DC-DC-STEP-DOWN-LM2596
- SV1: device con-lstb:MA03-1 -> con-lstb:MA06-1
Connections:
- new net 5V_PUI: CON_SERV1.2, CON_SERV2.2, CON_SERV3.2, U$3.OUT+
- new net N$10: Q1.G, R4.2, R5.1
- new net N$11: R5.2, U$1.36/A17
- new net N$12: D3.A, Q1.D, SL2.2
- new net N$13: SV3.2, U$1.17/A3
- new net N$14: ENCOD1.1, U$1.20/A6
- new net N$15: ENCOD1.2, U$1.21/A7
- new net N$16: CON_SERV2.1, U$1.15/A1
- new net N$17: CON_SERV3.1, U$1.37/A18
- new net N$18: DYNAMIX.3, U$1.32/A13
- new net N$19: CON_SERV1.1, U$1.39/A20
- new net N$2: CON_MOT2.3, U$1.29
- new net N$20: DYNAMIX.2, U$1.31/A12
- new net N$21: CON_I2C2_1.4, CON_I2C2_2.4, CON_I2C2_3.4, CON_I2C2_4.4, CON_I2C2_5.4, U$1.3/CANTX
- new net N$22: COULEUR.1, U$1.26
- new net N$23: CON_I2C2_1.3, CON_I2C2_2.3, CON_I2C2_3.3, CON_I2C2_4.3, CON_I2C2_5.3, U$1.4/CANRX
- new net N$24: DYNAMIX.1, U$1.30
- new net N$25: TIRETTE.1, U$1.25
- new net N$26: UART.2
- new net N$27: U$1.0/RX, UART.1
- new net N$3: CON_MOT1.3, U$1.5
- new net N$30: SV1.3, U$1.10/CS
- new net N$31: SV1.4, U$1.9/CS
- new net N$32: SV1.5, U$1.8
- new net N$33: SV1.6, U$1.7
- new net N$6: Q2.G, R2.2, R3.1
- new net N$7: R3.2, U$1.35/A16
- new net N$8: D2.A, Q2.D, SL1.2
- new net N$9: SV3.1, U$1.16/A2
- net 12V: now also D2.C, D3.C, SL1.1, SL2.1, U$3.IN+
- net 5V_SIG: now also CON_I2C2_1.1, CON_I2C2_2.1, CON_I2C2_3.1, CON_I2C2_4.1, CON_I2C2_5.1, DYNAMIX.5, ENCOD1.4, SV1.1, SV3.4
- net GND: now also CON_I2C2_1.2, CON_I2C2_2.2, CON_I2C2_3.2, CON_I2C2_4.2, CON_I2C2_5.2, CON_MOT1.1, CON_MOT2.1, CON_SERV1.3, CON_SERV2.3, CON_SERV3.3, COULEUR.2, DYNAMIX.4, ENCOD1.3, Q1.S, Q2.S, R2.1, R4.1, SV1.2, SV3.3, TIRETTE.2, U$3.IN-, U$3.OUT-, UART.3; no longer SV1.1, SV2.1
- net N$4: now also CON_MOT1.2, U$1.6; no longer SV1.2, U$1.2
- net N$5: now also CON_MOT2.2, U$1.28; no longer SV2.2, U$1.6

Commit message: [Secondary] Adds the board.
Parts:
- removed SL1, SL2: (no value), con-amp-quick:MA02
- added JP1, JP2: (no value), pinhead:PINHD-1X2
- Q1, Q2: value BUZ11 -> BUZ11BV; device transistor-fet:BUZ11 -> transistor-power:BUZ11BV
Connections:
- net 12V: now also JP1.1, JP2.1; no longer SL1.1, SL2.1
- net 5V_SIG: now also UART.4
- net N$12: now also JP1.2; no longer SL2.2
- net N$26: now also U$1.1/TX
- net N$8: now also JP2.2; no longer SL1.2
Changed lines of the file:
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@@
 <part name="CON_MOT2" library="con-lstb" deviceset="MA03-1" device=""/>
 <part name="SV3" library="con-lstb" deviceset="MA04-1" device=""/>
-<part name="Q2" library="transistor-fet" deviceset="BUZ11" device=""/>
+<part name="Q2" library="transistor-power" deviceset="BUZ11" device="BV"/>
 <part name="R2" library="resistor" deviceset="R-EU_" device="0204/7" value="10k"/>
 <part name="R3" library="resistor" deviceset="R-EU_" device="0204/7" value="10"/>
-<part name="SL1" library="con-amp-quick" deviceset="MA02" device=""/>
 <part name="D2" library="diode" deviceset="1N4004" device=""/>
-<part name="Q1" library="transistor-fet" deviceset="BUZ11" device=""/>
+<part name="Q1" library="transistor-power" deviceset="BUZ11" device="BV"/>
 <part name="R4" library="resistor" deviceset="R-EU_" device="0204/7" value="10k"/>
 <part name="R5" library="resistor" deviceset="R-EU_" device="0204/7" value="10"/>
-<part name="SL2" library="con-amp-quick" deviceset="MA02" device=""/>
 <part name="D3" library="diode" deviceset="1N4004" device=""/>
 <part name="ENCOD1" library="con-lstb" deviceset="MA04-1" device=""/>
@@
 <part name="UART" library="con-lstb" deviceset="MA04-1" device=""/>
 <part name="SV1" library="con-lstb" deviceset="MA06-1" device=""/>
+<part name="JP1" library="pinhead" deviceset="PINHD-1X2" device=""/>
+<part name="JP2" library="pinhead" deviceset="PINHD-1X2" device=""/>
 </parts>
 <sheets>
@@
 <instance part="CON_MOT2" gate="G$1" x="20.32" y="25.4"/>
 <instance part="SV3" gate="1" x="137.16" y="53.34" rot="MR0"/>
-<instance part="Q2" gate="G$1" x="152.4" y="-15.24"/>
+<instance part="Q2" gate="1" x="149.86" y="-12.7"/>
 <instance part="R2" gate="G$1" x="142.24" y="-25.4" rot="R90"/>
 <instance part="R3" gate="G$1" x="129.54" y="-17.78" rot="R180"/>
-<instance part="SL1" gate="G$1" x="177.8" y="-10.16" rot="R180"/>
 <instance part="D2" gate="1" x="187.96" y="-12.7" rot="R90"/>
-<instance part="Q1" gate="G$1" x="157.48" y="12.7"/>
+<instance part="Q1" gate="1" x="157.48" y="15.24"/>
 <instance part="R4" gate="G$1" x="147.32" y="2.54" rot="R90"/>
 <instance part="R5" gate="G$1" x="134.62" y="10.16" rot="R180"/>
-<instance part="SL2" gate="G$1" x="182.88" y="17.78" rot="R180"/>
 <instance part="D3" gate="1" x="193.04" y="15.24" rot="R90"/>
 <instance part="ENCOD1" gate="1" x="160.02" y="66.04" rot="MR0"/>
@@
 <instance part="UART" gate="1" x="38.1" y="86.36"/>
 <instance part="SV1" gate="1" x="-10.16" y="58.42"/>
+<instance part="JP1" gate="G$1" x="185.42" y="15.24"/>
+<instance part="JP2" gate="G$1" x="180.34" y="-12.7"/>
 </instances>
 <busses>
@@
 </segment>
 <segment>
-<pinref part="Q2" gate="G$1" pin="S"/>
-<wire x1="157.48" y1="-17.78" x2="160.02" y2="-17.78" width="0.1524" layer="91"/>
+<pinref part="Q2" gate="1" pin="S"/>
+<wire x1="152.4" y1="-17.78" x2="160.02" y2="-17.78" width="0.1524" layer="91"/>
 <label x="162.56" y="-20.32" size="1.778" layer="95"/>
 <pinref part="R2" gate="G$1" pin="1"/>
@@
 </segment>
 <segment>
-<pinref part="Q1" gate="G$1" pin="S"/>
-<wire x1="162.56" y1="10.16" x2="165.1" y2="10.16" width="0.1524" layer="91"/>
+<pinref part="Q1" gate="1" pin="S"/>
+<wire x1="160.02" y1="10.16" x2="165.1" y2="10.16" width="0.1524" layer="91"/>
 <label x="167.64" y="7.62" size="1.778" layer="95"/>
 <pinref part="R4" gate="G$1" pin="1"/>
@@
 </segment>
 <segment>
-<label x="160.02" y="-10.16" size="1.778" layer="95"/>
+<label x="154.94" y="-5.08" size="1.778" layer="95"/>
 <pinref part="D2" gate="1" pin="C"/>
-<wire x1="167.64" y1="-10.16" x2="157.48" y2="-10.16" width="0.1524" layer="91"/>
+<wire x1="167.64" y1="-5.08" x2="157.48" y2="-5.08" width="0.1524" layer="91"/>
 <wire x1="187.96" y1="-10.16" x2="187.96" y2="-2.54" width="0.1524" layer="91"/>
 <wire x1="187.96" y1="-2.54" x2="167.64" y2="-2.54" width="0.1524" layer="91"/>
-<wire x1="167.64" y1="-2.54" x2="167.64" y2="-10.16" width="0.1524" layer="91"/>
-<pinref part="SL1" gate="G$1" pin="1"/>
-<wire x1="167.64" y1="-10.16" x2="170.18" y2="-10.16" width="0.1524" layer="91"/>
-<junction x="167.64" y="-10.16"/>
-</segment>
-<segment>
-<label x="165.1" y="17.78" size="1.778" layer="95"/>
+<wire x1="167.64" y1="-2.54" x2="167.64" y2="-5.08" width="0.1524" layer="91"/>
+<junction x="167.64" y="-5.08"/>
+<pinref part="JP2" gate="G$1" pin="1"/>
+<wire x1="177.8" y1="-10.16" x2="170.18" y2="-10.16" width="0.1524" layer="91"/>
+<wire x1="170.18" y1="-10.16" x2="170.18" y2="-5.08" width="0.1524" layer="91"/>
+<wire x1="170.18" y1="-5.08" x2="167.64" y2="-5.08" width="0.1524" layer="91"/>
+</segment>
+<segment>
+<label x="162.56" y="22.86" size="1.778" layer="95"/>
 <pinref part="D3" gate="1" pin="C"/>
-<wire x1="172.72" y1="17.78" x2="162.56" y2="17.78" width="0.1524" layer="91"/>
+<wire x1="172.72" y1="22.86" x2="162.56" y2="22.86" width="0.1524" layer="91"/>
 <wire x1="193.04" y1="17.78" x2="193.04" y2="25.4" width="0.1524" layer="91"/>
 <wire x1="193.04" y1="25.4" x2="172.72" y2="25.4" width="0.1524" layer="91"/>
-<wire x1="172.72" y1="25.4" x2="172.72" y2="17.78" width="0.1524" layer="91"/>
-<pinref part="SL2" gate="G$1" pin="1"/>
-<wire x1="175.26" y1="17.78" x2="172.72" y2="17.78" width="0.1524" layer="91"/>
-<junction x="172.72" y="17.78"/>
+<wire x1="172.72" y1="25.4" x2="172.72" y2="22.86" width="0.1524" layer="91"/>
+<junction x="172.72" y="22.86"/>
+<pinref part="JP1" gate="G$1" pin="1"/>
+<wire x1="182.88" y1="17.78" x2="172.72" y2="17.78" width="0.1524" layer="91"/>
+<wire x1="172.72" y1="17.78" x2="172.72" y2="22.86" width="0.1524" layer="91"/>
 </segment>
 <segment>
@@
 </segment>
 <segment>
-<wire x1="43.18" y1="88.9" x2="53.34" y2="88.9" width="0.1524" layer="91"/>
 <label x="50.8" y="88.9" size="1.778" layer="95"/>
+<pinref part="UART" gate="1" pin="4"/>
+<wire x1="45.72" y1="88.9" x2="53.34" y2="88.9" width="0.1524" layer="91"/>
 </segment>
 <segment>
@@
 <segment>
 <pinref part="R3" gate="G$1" pin="1"/>
-<pinref part="Q2" gate="G$1" pin="G"/>
+<pinref part="Q2" gate="1" pin="G"/>
 <wire x1="134.62" y1="-17.78" x2="142.24" y2="-17.78" width="0.1524" layer="91"/>
 <pinref part="R2" gate="G$1" pin="2"/>
-<wire x1="142.24" y1="-17.78" x2="147.32" y2="-17.78" width="0.1524" layer="91"/>
+<wire x1="142.24" y1="-17.78" x2="144.78" y2="-17.78" width="0.1524" layer="91"/>
+<wire x1="144.78" y1="-17.78" x2="144.78" y2="-15.24" width="0.1524" layer="91"/>
+<wire x1="144.78" y1="-15.24" x2="147.32" y2="-15.24" width="0.1524" layer="91"/>
 <wire x1="142.24" y1="-20.32" x2="142.24" y2="-17.78" width="0.1524" layer="91"/>
 <junction x="142.24" y="-17.78"/>
@@
 <net name="N$8" class="0">
 <segment>
-<pinref part="Q2" gate="G$1" pin="D"/>
-<pinref part="SL1" gate="G$1" pin="2"/>
-<wire x1="157.48" y1="-12.7" x2="170.18" y2="-12.7" width="0.1524" layer="91"/>
+<pinref part="Q2" gate="1" pin="D"/>
+<wire x1="152.4" y1="-7.62" x2="162.56" y2="-7.62" width="0.1524" layer="91"/>
+<wire x1="162.56" y1="-7.62" x2="162.56" y2="-12.7" width="0.1524" layer="91"/>
+<wire x1="162.56" y1="-12.7" x2="170.18" y2="-12.7" width="0.1524" layer="91"/>
 <wire x1="170.18" y1="-12.7" x2="170.18" y2="-20.32" width="0.1524" layer="91"/>
 <pinref part="D2" gate="1" pin="A"/>
 <wire x1="170.18" y1="-20.32" x2="187.96" y2="-20.32" width="0.1524" layer="91"/>
 <wire x1="187.96" y1="-20.32" x2="187.96" y2="-15.24" width="0.1524" layer="91"/>
+<pinref part="JP2" gate="G$1" pin="2"/>
+<wire x1="177.8" y1="-12.7" x2="170.18" y2="-12.7" width="0.1524" layer="91"/>
+<junction x="170.18" y="-12.7"/>
 </segment>
 </net>
@@
 <segment>
 <pinref part="R5" gate="G$1" pin="1"/>
-<pinref part="Q1" gate="G$1" pin="G"/>
+<pinref part="Q1" gate="1" pin="G"/>
 <wire x1="139.7" y1="10.16" x2="147.32" y2="10.16" width="0.1524" layer="91"/>
 <pinref part="R4" gate="G$1" pin="2"/>
-<wire x1="147.32" y1="10.16" x2="152.4" y2="10.16" width="0.1524" layer="91"/>
+<wire x1="147.32" y1="10.16" x2="154.94" y2="10.16" width="0.1524" layer="91"/>
+<wire x1="154.94" y1="10.16" x2="154.94" y2="12.7" width="0.1524" layer="91"/>
 <wire x1="147.32" y1="7.62" x2="147.32" y2="10.16" width="0.1524" layer="91"/>
 <junction x="147.32" y="10.16"/>
@@
 <net name="N$12" class="0">
 <segment>
-<pinref part="Q1" gate="G$1" pin="D"/>
-<pinref part="SL2" gate="G$1" pin="2"/>
-<wire x1="162.56" y1="15.24" x2="175.26" y2="15.24" width="0.1524" layer="91"/>
+<pinref part="Q1" gate="1" pin="D"/>
+<wire x1="160.02" y1="20.32" x2="165.1" y2="20.32" width="0.1524" layer="91"/>
+<wire x1="165.1" y1="20.32" x2="165.1" y2="15.24" width="0.1524" layer="91"/>
+<wire x1="165.1" y1="15.24" x2="175.26" y2="15.24" width="0.1524" layer="91"/>
 <wire x1="175.26" y1="15.24" x2="175.26" y2="7.62" width="0.1524" layer="91"/>
 <pinref part="D3" gate="1" pin="A"/>
 <wire x1="175.26" y1="7.62" x2="193.04" y2="7.62" width="0.1524" layer="91"/>
 <wire x1="193.04" y1="7.62" x2="193.04" y2="12.7" width="0.1524" layer="91"/>
+<pinref part="JP1" gate="G$1" pin="2"/>
+<wire x1="182.88" y1="15.24" x2="175.26" y2="15.24" width="0.1524" layer="91"/>
+<junction x="175.26" y="15.24"/>
 </segment>
 </net>
@@
 <wire x1="45.72" y1="83.82" x2="50.8" y2="83.82" width="0.1524" layer="91"/>
 <wire x1="50.8" y1="83.82" x2="50.8" y2="68.58" width="0.1524" layer="91"/>
-<wire x1="50.8" y1="68.58" x2="66.04" y2="68.58" width="0.1524" layer="91"/>
-</segment>
-</net>
+<pinref part="U$1" gate="G$1" pin="1/TX"/>
+<wire x1="50.8" y1="68.58" x2="63.5" y2="68.58" width="0.1524" layer="91"/>
+</segment>
+</net>

Commit message: [secondary] Adds the final board
Parts:
- removed C1, C2: (no value), rcl:C-EU025-060X050
- removed D1: 1N4004, diode:1N4004
- removed R1: 348, resistor:R-EU_0204/7
- removed U$2: PTH08080, pth08080:PTH08080
- added U1: TSR_1-2450, SamacSys_Parts:TSR_1-2450
Connections:
- removed net N$1: R1.2, U$2.ADJ
- net 12V: now also U1.VIN+; no longer C2.2, D1.C, U$2.VIN
- net 5V_SIG: now also U1.VOUT+; no longer C1.1, D1.A, U$2.VOUT
- net GND: now also U1.GND; no longer C1.2, C2.1, R1.1, U$2.GND
Changed lines of the file:
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@@
 <?xml version="1.0" encoding="utf-8"?>
 <!DOCTYPE eagle SYSTEM "eagle.dtd">
-<eagle version="6.1">
+<eagle version="8.6.0">
 <drawing>
 <settings>
 <setting alwaysvectorfont="no"/>
+<setting keepoldvectorfont="yes"/>
 <setting verticaltext="up"/>
 </settings>
@@
 <parts>
 <part name="U$1" library="Teensy356" deviceset="TEENSY_3.5/3.6" device=""/>
-<part name="U$2" library="pth08080" deviceset="PTH08080" device=""/>
-<part name="R1" library="resistor" deviceset="R-EU_" device="0204/7" value="348"/>
-<part name="C1" library="rcl" deviceset="C-EU" device="025-060X050"/>
-<part name="C2" library="rcl" deviceset="C-EU" device="025-060X050"/>
-<part name="D1" library="diode" deviceset="1N4004" device=""/>
 <part name="BAT" library="con-ptr500" deviceset="AK300/2" device=""/>
 <part name="CON_MOT1" library="con-lstb" deviceset="MA03-1" device=""/>
@@
 <part name="JP1" library="pinhead" deviceset="PINHD-1X2" device=""/>
 <part name="JP2" library="pinhead" deviceset="PINHD-1X2" device=""/>
+<part name="U1" library="SamacSys_Parts" deviceset="TSR_1-2450" device=""/>
 </parts>
 <sheets>
@@
 <instances>
 <instance part="U$1" gate="G$1" x="83.82" y="60.96"/>
-<instance part="U$2" gate="G$1" x="-38.1" y="137.16"/>
-<instance part="R1" gate="G$1" x="-25.4" y="127" rot="R90"/>
-<instance part="C1" gate="G$1" x="-17.78" y="134.62"/>
-<instance part="C2" gate="G$1" x="-58.42" y="129.54" rot="R180"/>
-<instance part="D1" gate="1" x="-40.64" y="154.94" rot="R180"/>
 <instance part="BAT" gate="-1" x="-88.9" y="139.7"/>
 <instance part="BAT" gate="-2" x="-88.9" y="134.62"/>
@@
 <instance part="JP1" gate="G$1" x="185.42" y="15.24"/>
 <instance part="JP2" gate="G$1" x="180.34" y="-12.7"/>
+<instance part="U1" gate="G$1" x="-40.64" y="137.16"/>
 </instances>
 <busses>
 </busses>
 <nets>
-<net name="N$1" class="0">
-<segment>
-<pinref part="U$2" gate="G$1" pin="ADJ"/>
-<pinref part="R1" gate="G$1" pin="2"/>
-<wire x1="-30.48" y1="132.08" x2="-25.4" y2="132.08" width="0.1524" layer="91"/>
-</segment>
-</net>
 <net name="GND" class="0">
 <segment>
-<pinref part="R1" gate="G$1" pin="1"/>
-<pinref part="U$2" gate="G$1" pin="GND"/>
-<wire x1="-25.4" y1="121.92" x2="-40.64" y2="121.92" width="0.1524" layer="91"/>
-<wire x1="-40.64" y1="127" x2="-40.64" y2="121.92" width="0.1524" layer="91"/>
-<pinref part="C1" gate="G$1" pin="2"/>
-<wire x1="-17.78" y1="129.54" x2="-17.78" y2="121.92" width="0.1524" layer="91"/>
-<wire x1="-17.78" y1="121.92" x2="-25.4" y2="121.92" width="0.1524" layer="91"/>
-<junction x="-25.4" y="121.92"/>
-<pinref part="C2" gate="G$1" pin="1"/>
-<wire x1="-58.42" y1="127" x2="-58.42" y2="121.92" width="0.1524" layer="91"/>
-<wire x1="-58.42" y1="121.92" x2="-40.64" y2="121.92" width="0.1524" layer="91"/>
-<junction x="-40.64" y="121.92"/>
 <pinref part="BAT" gate="-2" pin="KL"/>
 <wire x1="-83.82" y1="134.62" x2="-71.12" y2="134.62" width="0.1524" layer="91"/>
 <wire x1="-71.12" y1="134.62" x2="-71.12" y2="121.92" width="0.1524" layer="91"/>
-<wire x1="-71.12" y1="121.92" x2="-58.42" y2="121.92" width="0.1524" layer="91"/>
-<junction x="-58.42" y="121.92"/>
+<pinref part="U1" gate="G$1" pin="GND"/>
+<wire x1="-40.64" y1="134.62" x2="-45.72" y2="134.62" width="0.1524" layer="91"/>
+<wire x1="-71.12" y1="121.92" x2="-45.72" y2="121.92" width="0.1524" layer="91"/>
+<wire x1="-45.72" y1="121.92" x2="-45.72" y2="134.62" width="0.1524" layer="91"/>
+<label x="-45.72" y="129.54" size="1.778" layer="95"/>
 </segment>
 <segment>
@@
 <net name="12V" class="0">
 <segment>
-<pinref part="U$2" gate="G$1" pin="VIN"/>
-<pinref part="C2" gate="G$1" pin="2"/>
-<wire x1="-48.26" y1="139.7" x2="-58.42" y2="139.7" width="0.1524" layer="91"/>
-<wire x1="-58.42" y1="139.7" x2="-58.42" y2="134.62" width="0.1524" layer="91"/>
-<wire x1="-58.42" y1="139.7" x2="-58.42" y2="149.86" width="0.1524" layer="91"/>
-<junction x="-58.42" y="139.7"/>
-<label x="-66.04" y="139.7" size="1.778" layer="95"/>
-<pinref part="D1" gate="1" pin="C"/>
-<wire x1="-43.18" y1="154.94" x2="-58.42" y2="154.94" width="0.1524" layer="91"/>
-<wire x1="-58.42" y1="154.94" x2="-58.42" y2="139.7" width="0.1524" layer="91"/>
-<wire x1="-58.42" y1="139.7" x2="-63.5" y2="139.7" width="0.1524" layer="91"/>
-<pinref part="BAT" gate="-1" pin="KL"/>
-<wire x1="-63.5" y1="139.7" x2="-66.04" y2="139.7" width="0.1524" layer="91"/>
-<wire x1="-83.82" y1="139.7" x2="-66.04" y2="139.7" width="0.1524" layer="91"/>
-</segment>
-<segment>
 <label x="154.94" y="-5.08" size="1.778" layer="95"/>
 <pinref part="D2" gate="1" pin="C"/>
@@
 <label x="53.34" y="139.7" size="1.778" layer="95"/>
 </segment>
+<segment>
+<pinref part="U1" gate="G$1" pin="VIN+"/>
+<label x="-45.72" y="137.16" size="1.778" layer="95"/>
+<pinref part="BAT" gate="-1" pin="KL"/>
+<wire x1="-40.64" y1="137.16" x2="-83.82" y2="137.16" width="0.1524" layer="91"/>
+<wire x1="-83.82" y1="137.16" x2="-83.82" y2="139.7" width="0.1524" layer="91"/>
+</segment>
 </net>
 <net name="5V_SIG" class="0">
-<segment>
-<pinref part="U$2" gate="G$1" pin="VOUT"/>
-<pinref part="C1" gate="G$1" pin="1"/>
-<wire x1="-30.48" y1="139.7" x2="-17.78" y2="139.7" width="0.1524" layer="91"/>
-<wire x1="-17.78" y1="139.7" x2="-17.78" y2="137.16" width="0.1524" layer="91"/>
-<wire x1="-17.78" y1="139.7" x2="-5.08" y2="139.7" width="0.1524" layer="91"/>
-<junction x="-17.78" y="139.7"/>
-<label x="-2.54" y="139.7" size="1.778" layer="95"/>
-<pinref part="D1" gate="1" pin="A"/>
-<wire x1="-17.78" y1="139.7" x2="-17.78" y2="154.94" width="0.1524" layer="91"/>
-<wire x1="-17.78" y1="154.94" x2="-38.1" y2="154.94" width="0.1524" layer="91"/>
-</segment>
 <segment>
 <pinref part="U$1" gate="G$1" pin="VIN"/>
@@
 <wire x1="-2.54" y1="50.8" x2="0" y2="50.8" width="0.1524" layer="91"/>
 <label x="0" y="50.8" size="1.778" layer="95"/>
+</segment>
+<segment>
+<pinref part="U1" gate="G$1" pin="VOUT+"/>
+<wire x1="-10.16" y1="137.16" x2="-5.08" y2="137.16" width="0.1524" layer="91"/>
+<label x="-5.08" y="137.16" size="1.778" layer="95"/>
 </segment>
 </net>
@@
 </schematic>
 </drawing>
+<compatibility>
+<note version="6.3" minversion="6.2.2" severity="warning">
+Since Version 6.2.2 text objects can contain more than one line,
+which will not be processed correctly with this version.
+</note>
+</compatibility>
 </eagle>
