File: 2018/FAT2/fat2.sch (EAGLE design)
At the start: 30 parts, among them Q1 BUZ11BV, Q2 BUZ11BV, U1 TSR_1-2450, U2 TSR_1-2450, U3 TSR_1-2433

Commit message: [FAT V2] Route easy side.
Parts:
- removed JP3, JP4: (no value), pinhead:PINHD-1X4
- added DYNUART: (no value), pinhead:PINHD-1X5
- added I2C1, UART4: (no value), pinhead:PINHD-1X4
- added M4: (no value), pinhead:PINHD-1X3
- R3, R4, R5, R6: value 10k -> (none); device rcl:R-EU_0204/7 -> rcl:R-EU_R0805
- renumbered JP1 to UART1, JP2 to UART2, U1 to RG5V_SIG, U2 to RG5V_POW, U3 to RG3V3
Connections:
- removed net N$10: UART2.1
- removed net N$11: UART2.2
- removed net N$12: UART2.3
- removed net N$13: UART2.4
- new net 29: M4.3, U$1.29
- new net 30: M4.2, U$1.30
- new net DYN_CTRL: DYNUART.5, U$1.35/A16
- new net N$6: U$1.17/A3
- new net RX2: U$1.9/CS, UART2.4
- new net RX4: U$1.31/A12, UART4.4
- new net RX5: DYNUART.4, U$1.34/A15
- new net SCL1: I2C1.4, U$1.37/A18
- new net SDA1: I2C1.3, U$1.38/A19
- new net TX2: U$1.10/CS, UART2.3
- new net TX4: U$1.32/A13, UART4.3
- new net TX5: DYNUART.3, U$1.33/A14
- net 5V_SIG: now also DYNUART.1, I2C1.1, UART2.1, UART4.1
- net DIR1: now also U$1.3/CANTX
- net DIR2: now also U$1.5
- net DIR3: now also U$1.7
- net ENC_1_A: now also U$1.11/MOSI
- net ENC_1_B: now also U$1.12/MISO
- net ENC_2_A: now also U$1.24
- net ENC_2_B: now also U$1.25
- net ENC_3_A: now also U$1.26
- net ENC_3_B: now also U$1.27
- net GND: now also DYNUART.2, I2C1.2, M4.1, UART2.2, UART4.2
- net MOT1: now also U$1.22/A8
- net MOT2: now also U$1.23/A9
- net POW_LEVEL: now also U$1.A22/DAC1
- net PWM1: now also U$1.2
- net PWM2: now also U$1.4/CANRX
- net PWM3: now also U$1.6
- net SERVO1: now also U$1.16/A2
- net SERVO2: now also U$1.15/A1
- net SERVO3: now also U$1.14/A0
- net SIG_LEVEL: now also U$1.A21/DAC0

Commit message: [FAT V2] Finish board.
Parts:
- removed R3, R4, R5, R6: (no value), rcl:R-EU_R0805
- added JP1: (no value), pinhead:PINHD-1X2/90
- added R10, R7, R8, R9: 10k, rcl:R-EU_0204/7
- added SPARE: (no value), pinhead:PINHD-1X5
Connections:
- new net GND2: R10.1, R8.1, U$1.GND2
- new net N$1: SPARE.5, U$1.17/A3
- new net N$2: SPARE.4, U$1.18/A4/SDA
- new net N$4: SPARE.3, U$1.19/A5/SCL
- new net N$8: SPARE.1, U$1.21/A7
- net 12V_POW: now also R7.2; no longer R4.2
- net 12V_SIG: now also R9.2; no longer R5.2
- net 5V_SIG: now also JP1.1, U$1.VIN
- net GND: now also Q1.S, Q2.S, R1.1, R2.1; no longer R3.1, R6.1
- net N$6: now also SPARE.2, U$1.20/A6; no longer U$1.17/A3
- net N$7: now also JP1.2, U$1.VUSB; no longer Q1.S, Q2.S, R1.1, R2.1
- net POW_LEVEL: now also R7.1, R8.2; no longer R3.2, R4.1
- net SIG_LEVEL: now also R10.2, R9.1; no longer R5.1, R6.2
