File: 2018/robot_base/robot_base/robot_systems.sch (EAGLE design)
At the start: 41 parts, among them IC1 DRV8840PWP, IC2 DRV8840PWP, IC3 DRV8840PWP

Commit message: Update robot_system.sch/brd: Minor corrections in sch and start to route.
Parts:
- removed BAU_BAT1, BAU_BAT2: (no value), con-ptr500:AK500/2
- removed I2C0, I2C1, I2C2, JP10, JP_CUR1, JP_CUR2, JP_CUR3, JP_MOT1, JP_MOT2, JP_MOT3: (no value), pinhead:PINHD-1X4
- removed JP_I2C0_VCC, JP_I2C1_VCC, JP_I2C2_VCC: (no value), pinhead:PINHD-1X1
- removed R1, R2, R3: (no value), rcl:R-EU_0204/5
- added I2C3, I2C4, I2C5, JP8: (no value), pinhead:PINHD-1X4
- added IC1_C1, IC2_C1, IC3_C1: 0.01uF, rcl:C-EUC0603
- added IC1_C2, IC1_C3, IC2_C2, IC2_C3, IC2_C4, IC3_C2, IC3_C3, IC3_C4: 0.1uF, SparkFun-Passives:CAP0805
- added IC1_C4: 0.1uF, SparkFun-Passives:CAP1206
- added IC1_C5, IC2_C5, IC3_C5: 100uF, SparkFun-Passives:CAP_POL3528-KIT
- added IC1_C6, IC2_C6, IC3_C6: 470nF, rcl:C-EUC0603
- added IC1_R1, IC1_R2, IC2_R1, IC2_R2, IC3_R1, IC3_R2: ???, resistor:R-EU_0204/5
- added IC1_R3, IC2_R3, IC3_R3: 10k, rcl:R-EU_R2010
- added IC1_R4, IC2_R4, IC3_R4: 100m, rcl:R-EU_R2512
- added IC1_R5, IC2_R5, IC3_R5: 1M, rcl:R-EU_R0603
- added J1: (no value), SparkFun-Connectors:M02PTH
- added JP1, JP13, JP14, JP15, JP16, JP17, JP18, JP19, JP2, JP20, JP21, JP22, JP23, JP3, JP4, JP5, JP6, JP9: (no value), pinhead:PINHD-1X2
- added JP7: (no value), adafruit:PINHD-1X3
- added JP_I2C0_VCC1, JP_I2C1_VCC1, JP_I2C2_VCC1: (no value), pinhead:PINHD-1X3
- added M1, M2, M3: (no value), con-ptr500:AK500/2
- added R4, R5, R6, R7, R8, R9: (no value), rcl:R-EU_0204/5
- U$1: value TEENSY_3.5/3.6 -> TEENSY_3.5/3.6TEENSY_3.5/3.6_LONG_PADS; device Teensy356:TEENSY_3.5/3.6 -> Teensy356:TEENSY_3.5/3.6TEENSY_3.5/3.6_LONG_PADS
Connections:
- removed net 3V3_TEESNY_1: U$1.3V3_LO
- removed net 3V3_TEESNY_2: JP10.3, U$1.3V3
- removed net CUR3_SE: JP_CUR3.2, U$1.39/A20
- removed net MOT1_IN_A: JP_MOT1.1, U$1.8
- removed net MOT1_IN_B: JP_MOT1.2, U$1.23/A9
- removed net MOT2_IN_A: JP_MOT2.1, U$1.9/CS
- removed net MOT2_IN_B: JP_MOT2.2, U$1.22/A8
- removed net MOT3_IN_A: JP_MOT3.1, U$1.10/CS
- removed net MOT3_IN_B: JP_MOT3.2, U$1.21/A7
- removed net N$28: U$1.U5V
- removed net N$29: U$1.UD-
- removed net N$30: U$1.UD+
- removed net N$31: U$1.UGND1
- removed net N$32: U$1.UGND2
- removed net N$33: U$1.A11
- removed net N$34: U$1.A10
- removed net N$35: U$1.AREF
- removed net N$36: U$1.VUSB
- removed net N$61: U$1.RESET
- removed net N$62: U$1.PROG
- removed net N$63: U$1.GND3
- removed net N$64: U$1.3V3_2
- removed net N$65: U$1.VBAT
- new net 12V2: 12V_PWR_1-1.KL, 12V_PWR_2-1.KL, 12V_PWR_3-1.KL, BAT_2-1.KL, IC1.VM(1), IC1.VM(2), IC1_C2.1, IC1_C3.2, IC1_C4.2, IC1_C5.+, IC1_R5.1, IC2.VM(1), IC2.VM(2), IC2_C2.1, IC2_C3.2, IC2_C4.2, IC2_C5.+, IC2_R5.1, IC3.VM(1), IC3.VM(2), IC3_C2.1, IC3_C3.2, IC3_C4.2, IC3_C5.+, IC3_R5.1
- new net IC1_I0: IC1.I0, JP1.2
- new net IC1_I1: IC1.I1, JP2.2
- new net IC1_I2: IC1.I2, JP3.2
- new net IC1_I3: IC1.I3, JP4.2
- new net IC1_I4: IC1.I4, JP5.2
- new net IC1_NFAULT: IC1.NFAULT, IC1_R3.1, U$1.2
- new net IC1_NRESET: IC1.NRESET, JP6.2
- new net IC1_NSLEEP: IC1.NSLEEP, JP6.1
- new net IC1_V3P3: IC1.DECAY, IC1.V3P3OUT, IC1_C6.1, IC1_R1.1, IC1_R3.2
- new net IC2_I0: IC2.I0, JP9.2
- new net IC2_I1: IC2.I1, JP13.2
- new net IC2_I2: IC2.I2, JP14.2
- new net IC2_I3: IC2.I3, JP15.2
- new net IC2_I4: IC2.I4, JP16.2
- new net IC2_NFAULT: IC2.NFAULT, IC2_R3.1, U$1.7
- new net IC2_NRESET: IC2.NRESET, JP17.2
- new net IC2_NSLEEP: IC2.NSLEEP, JP17.1
- new net IC2_V3P3: IC2.DECAY, IC2.V3P3OUT, IC2_C6.1, IC2_R1.1, IC2_R3.2
- new net IC3_I0: IC3.I0, JP18.2
- new net IC3_I1: IC3.I1, JP19.2
- new net IC3_I2: IC3.I2, JP20.2
- new net IC3_I3: IC3.I3, JP21.2
- new net IC3_I4: IC3.I4, JP22.2
- new net IC3_NFAULT: IC3.NFAULT, IC3_R3.1, U$1.10/CS
- new net IC3_NRESET: IC3.NRESET, JP23.2
- new net IC3_NSLEEP: IC3.NSLEEP, JP23.1
- new net IC3_R2: IC3.VREF(1), IC3.VREF(2), IC3_R1.2, IC3_R2.2
- new net IC3_V3P3: IC3.DECAY, IC3.V3P3OUT, IC3_C6.1, IC3_R1.1, IC3_R3.2
- new net M1_1: IC1.OUT1(1), IC1.OUT1(2), M1-1.KL
- new net M1_2: IC1.OUT2(1), IC1.OUT2(2), M1-2.KL
- new net M2_1: IC2.OUT1(1), IC2.OUT1(2), M2-1.KL
- new net M2_2: IC2.OUT2(1), IC2.OUT2(2), M2-2.KL
- new net M3_1: IC3.OUT1(1), IC3.OUT1(2), M3-1.KL
- new net M3_2: IC3.OUT2(1), IC3.OUT2(2), M3-2.KL
- new net MOT1_DIR: IC1.PHASE, U$1.5
- new net MOT2_DIR: IC2.PHASE, U$1.8
- new net MOT3_DIR: IC3.PHASE, U$1.29
- new net N$12: IC1.VCP, IC1_C2.2, IC1_R5.2
- new net N$13: IC2.CP2(1), IC2_C1.1
- new net N$14: IC2.CP2(2), IC2_C1.2
- new net N$15: IC2.VCP, IC2_C2.2, IC2_R5.2
- new net N$17: IC3.ISEN(1), IC3.ISEN(2), IC3_R4.2
- new net N$18: IC3.CP2(1), IC3_C1.1
- new net N$19: IC3.CP2(2), IC3_C1.2
- new net N$20: IC3.VCP, IC3_C2.2, IC3_R5.2
- new net NS50: JP7.3, U$1.39/A20
- net 3V3: now also JP1.1, JP13.1, JP14.1, JP15.1, JP16.1, JP18.1, JP19.1, JP2.1, JP20.1, JP21.1, JP22.1, JP3.1, JP4.1, JP5.1, JP9.1, JP_I2C0_VCC1.3, JP_I2C1_VCC1.3, JP_I2C2_VCC1.3
- net 5V: now also JP_I2C0_VCC1.1, JP_I2C1_VCC1.1, JP_I2C2_VCC1.1; no longer JP_CUR1.3, JP_CUR2.3, JP_CUR3.3
- net CUR1_NF: now also JP11.1; no longer JP_CUR1.1
- net CUR1_SE: now also JP8.4; no longer JP_CUR1.2
- net CUR2_NF: now also JP8.3; no longer JP_CUR2.1
- net CUR2_SE: now also JP8.2; no longer JP_CUR2.2
- net CUR3_NF: now also JP8.1; no longer JP_CUR3.1
- net ENC1_A: now also U$1.12/MISO; no longer U$1.25
- net ENC1_B: now also U$1.24; no longer U$1.26
- net ENC2_A: now also U$1.25; no longer U$1.27
- net ENC2_B: now also U$1.26; no longer U$1.28
- net ENC3_A: now also U$1.27; no longer U$1.29
- net ENC3_B: now also U$1.28; no longer U$1.30
- net GND: now also I2C3.2, I2C4.2, I2C5.2, IC1.GND(1), IC1.GND(2), IC1.THERMAL_PAD, IC1_C3.1, IC1_C4.1, IC1_C5.-, IC1_C6.2, IC1_R2.1, IC1_R4.1, IC2.GND(1), IC2.GND(2), IC2.THERMAL_PAD, IC2_C3.1, IC2_C4.1, IC2_C5.-, IC2_C6.2, IC2_R2.1, IC2_R4.1, IC3.GND(1), IC3.GND(2), IC3.THERMAL_PAD, IC3_C3.1, IC3_C4.1, IC3_C5.-, IC3_C6.2, IC3_R2.1, IC3_R4.1; no longer I2C0.2, I2C1.2, I2C2.2, JP_CUR1.4, JP_CUR2.4, JP_CUR3.4, JP_MOT1.4, JP_MOT2.4, JP_MOT3.4
- net I2C0_VCC: now also I2C3.1, JP_I2C0_VCC1.2, R4.1, R5.2; no longer I2C0.1, R1.1
- net I2C1_VCC: now also I2C4.1, JP_I2C1_VCC1.2, R6.1, R7.2; no longer I2C1.1, R2.1
- net I2C2_VCC: now also I2C5.1, JP_I2C2_VCC1.2, R8.1, R9.2; no longer I2C2.1, R3.1
- net MOT1_PWM: now also IC1.ENBL, U$1.6; no longer JP_MOT1.3, U$1.5
- net MOT2_PWM: now also IC2.ENBL, U$1.9/CS; no longer JP_MOT2.3, U$1.6
- net MOT3_PWM: now also IC3.ENBL, U$1.30; no longer JP_MOT3.3, U$1.7
- net N$1: now also JP11.4, U$1.23/A9; no longer JP10.1, U$1.11/MOSI
- net N$10: now also IC1.CP2(1), IC1_C1.1; no longer JP_I2C1_VCC.1, R2.2
- net N$11: now also IC1.CP2(2), IC1_C1.2; no longer JP_I2C2_VCC.1, R3.2
- net N$2: now also IC1.VREF(1), IC1.VREF(2), IC1_R1.2, IC1_R2.2; no longer 12V_PWR_1-1.KL, 12V_PWR_2-1.KL, 12V_PWR_3-1.KL, BAU_BAT2-2.KL
- net N$3: now also IC2.VREF(1), IC2.VREF(2), IC2_R1.2, IC2_R2.2; no longer BAT_2-1.KL, BAU_BAT2-1.KL
- net N$4: now also JP11.3, U$1.22/A8; no longer JP10.2, U$1.12/MISO
- net N$5: now also IC1.ISEN(1), IC1.ISEN(2), IC1_R4.2; no longer BAU_BAT1-1.KL, D24V22F3.VIN, D24V50F5.VIN
- net N$52: now also JP7.1; no longer JP11.4
- net N$53: now also JP7.2; no longer JP11.3
- net N$57: now also J1.1; no longer JP11.2
- net N$58: now also J1.2; no longer JP11.1
- net N$6: now also JP11.2, U$1.21/A7; no longer JP10.4, U$1.24
- net N$7: now also U$1.11/MOSI; no longer U$1.2
- net N$8: now also D24V22F3.VIN, D24V50F5.VIN; no longer BAU_BAT1-2.KL
- net N$9: now also IC2.ISEN(1), IC2.ISEN(2), IC2_R4.2; no longer JP_I2C0_VCC.1, R1.2
- net SCL0: now also I2C3.3, R4.2; no longer I2C0.3
- net SCL1: now also I2C4.3, R6.2; no longer I2C1.3
- net SCL2: now also I2C5.3, R8.2; no longer I2C2.3
- net SDA0: now also I2C3.4, R5.1; no longer I2C0.4
- net SDA1: now also I2C4.4, R7.1; no longer I2C1.4
- net SDA2: now also I2C5.4, R9.1; no longer I2C2.4
Other:
- moved on the sheet: IC1, IC2, IC3, JP11, JP12

Commit message: Update and complete routing of robot_system board. Last checks TODO.
Parts:
- removed I2C5: (no value), pinhead:PINHD-1X4
- added I2C2: (no value), pinhead:PINHD-1X4
- IC2_C4, IC3_C4: device SparkFun-Passives:CAP0805 -> SparkFun-Passives:CAP1206
- renumbered I2C3 to I2C0, I2C4 to I2C1, JP1 to JP1_I0, JP13 to JP2_I1, JP14 to JP2_I2, JP15 to JP2_I3, JP16 to JP2_I4, JP17 to JP2_S, JP18 to JP3_I0, JP19 to JP3_I1, JP2 to JP1_I1, JP20 to JP3_I2, JP21 to JP3_I3, JP22 to JP3_I4, JP23 to JP3_S, JP3 to JP1_I2, JP4 to JP1_I3, JP5 to JP1_I4, JP6 to JP1_S, JP9 to JP2_I0
Connections:
- net GND: now also I2C2.2; no longer I2C5.2
- net I2C2_VCC: now also I2C2.1; no longer I2C5.1
- net SCL2: now also I2C2.3; no longer I2C5.3
- net SDA2: now also I2C2.4; no longer I2C5.4
Other:
- moved on the sheet: JP_I2C2_VCC1, R8, R9

Commit message: [robot_system] Increase clearance, update package of one condo
Parts:
- IC1_C5, IC2_C5, IC3_C5: device SparkFun-Passives:CAP_POL3528-KIT -> SparkFun-Passives:CAP_POL7343
Changed lines of the file:
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@@
 <part name="IC1_C3" library="SparkFun-Passives" deviceset="CAP" device="0805" value="0.1uF"/>
 <part name="IC1_C4" library="SparkFun-Passives" deviceset="CAP" device="1206" value="0.1uF"/>
-<part name="IC1_C5" library="SparkFun-Passives" deviceset="CAP_POL" device="3528-KIT" value="100uF"/>
+<part name="IC1_C5" library="SparkFun-Passives" deviceset="CAP_POL" device="7343" value="100uF"/>
 <part name="IC1_R3" library="rcl" deviceset="R-EU_" device="R2010" value="10k"/>
 <part name="IC1_C6" library="rcl" deviceset="C-EU" device="C0603" value="470nF"/>
@@
 <part name="IC2_C3" library="SparkFun-Passives" deviceset="CAP" device="0805" value="0.1uF"/>
 <part name="IC2_C4" library="SparkFun-Passives" deviceset="CAP" device="1206" value="0.1uF"/>
-<part name="IC2_C5" library="SparkFun-Passives" deviceset="CAP_POL" device="3528-KIT" value="100uF"/>
+<part name="IC2_C5" library="SparkFun-Passives" deviceset="CAP_POL" device="7343" value="100uF"/>
 <part name="IC2_R3" library="rcl" deviceset="R-EU_" device="R2010" value="10k"/>
 <part name="IC2_C6" library="rcl" deviceset="C-EU" device="C0603" value="470nF"/>
@@
 <part name="IC3_C3" library="SparkFun-Passives" deviceset="CAP" device="0805" value="0.1uF"/>
 <part name="IC3_C4" library="SparkFun-Passives" deviceset="CAP" device="1206" value="0.1uF"/>
-<part name="IC3_C5" library="SparkFun-Passives" deviceset="CAP_POL" device="3528-KIT" value="100uF"/>
+<part name="IC3_C5" library="SparkFun-Passives" deviceset="CAP_POL" device="7343" value="100uF"/>
 <part name="IC3_R3" library="rcl" deviceset="R-EU_" device="R2010" value="10k"/>
 <part name="IC3_C6" library="rcl" deviceset="C-EU" device="C0603" value="470nF"/>

Commit message: Debut test motor control
Parts:
- removed 12V_PWR_1, 12V_PWR_2, 12V_PWR_3, BAT_1, BAT_2, M2, M3: (no value), con-ptr500:AK500/2
- removed D24V22F3: D24V22F3, D24V22F3:D24V22F3
- removed D24V50F5: D24V50F5, D24V50F5:D24V50F5
- removed I2C0, I2C1, I2C2, JP11, JP8, JP_ENC1, JP_ENC2, JP_ENC3, JP_UART1, JP_UART4, JP_UART5: (no value), pinhead:PINHD-1X4
- removed IC2, IC3: DRV8840PWP, DRV8840PWP:DRV8840PWP
- removed IC2_C1, IC3_C1: 0.01uF, rcl:C-EUC0603
- removed IC2_C2, IC2_C3, IC3_C2, IC3_C3: 0.1uF, SparkFun-Passives:CAP0805
- removed IC2_C4, IC3_C4: 0.1uF, SparkFun-Passives:CAP1206
- removed IC2_C5, IC3_C5: 100uF, SparkFun-Passives:CAP_POL7343
- removed IC2_C6, IC3_C6: 470nF, rcl:C-EUC0603
- removed IC2_R1, IC2_R2, IC3_R1, IC3_R2: ???, resistor:R-EU_0204/5
- removed IC2_R3, IC3_R3: 10k, rcl:R-EU_R2010
- removed IC2_R4, IC3_R4: 100m, rcl:R-EU_R2512
- removed IC2_R5, IC3_R5: 1M, rcl:R-EU_R0603
- removed J1: (no value), SparkFun-Connectors:M02PTH
- removed JP12: (no value), pinhead:PINHD-1X1
- removed JP1_I0, JP1_I1, JP1_I2, JP1_I3, JP1_I4, JP1_S, JP2_I0, JP2_I1, JP2_I2, JP2_I3, JP2_I4, JP2_S, JP3_I0, JP3_I1, JP3_I2, JP3_I3, JP3_I4, JP3_S: (no value), pinhead:PINHD-1X2
- removed JP7: (no value), adafruit:PINHD-1X3
- removed JP_3V3, JP_5V: (no value), pinhead:PINHD-2X4
- removed JP_I2C0_VCC1, JP_I2C1_VCC1, JP_I2C2_VCC1: (no value), pinhead:PINHD-1X3
- removed R4, R5, R6, R7, R8, R9: (no value), rcl:R-EU_0204/5
- removed U$1: TEENSY_3.5/3.6TEENSY_3.5/3.6_LONG_PADS, Teensy356:TEENSY_3.5/3.6TEENSY_3.5/3.6_LONG_PADS
- removed X_3V3: (no value), con-ptr500:AK300/4
- removed X_5V: (no value), con-ptr500:AK300/6
- added JP1: (no value), pinhead:PINHD-1X6
- added JP2: (no value), pinhead:PINHD-1X4
- added JP3: (no value), pinhead:PINHD-1X3
Connections:
- removed net 3V3: D24V22F3.VOUT, JP1_I0.1, JP1_I1.1, JP1_I2.1, JP1_I3.1, JP1_I4.1, JP2_I0.1, JP2_I1.1, JP2_I2.1, JP2_I3.1, JP2_I4.1, JP3_I0.1, JP3_I1.1, JP3_I2.1, JP3_I3.1, JP3_I4.1, JP_3V3.1, JP_3V3.3, JP_3V3.5, JP_3V3.7, JP_I2C0_VCC1.3, JP_I2C1_VCC1.3, JP_I2C2_VCC1.3, X_3V3-1.KL, X_3V3-3.KL
- removed net 5V: D24V50F5.OUT, JP_5V.1, JP_5V.3, JP_5V.5, JP_5V.7, JP_ENC1.2, JP_ENC2.2, JP_ENC3.2, JP_I2C0_VCC1.1, JP_I2C1_VCC1.1, JP_I2C2_VCC1.1, U$1.VIN, X_5V-1.KL, X_5V-3.KL, X_5V-5.KL
- removed net CUR1_NF: JP11.1, U$1.20/A6
- removed net CUR1_SE: JP8.4, U$1.17/A3
- removed net CUR2_NF: JP8.3, U$1.16/A2
- removed net CUR2_SE: JP8.2, U$1.15/A1
- removed net CUR3_NF: JP8.1, U$1.14/A0
- removed net ENC1_A: JP_ENC1.3, U$1.12/MISO
- removed net ENC1_B: JP_ENC1.4, U$1.24
- removed net ENC2_A: JP_ENC2.3, U$1.25
- removed net ENC2_B: JP_ENC2.4, U$1.26
- removed net ENC3_A: JP_ENC3.3, U$1.27
- removed net ENC3_B: JP_ENC3.4, U$1.28
- removed net I2C0_VCC: I2C0.1, JP_I2C0_VCC1.2, R4.1, R5.2
- removed net I2C1_VCC: I2C1.1, JP_I2C1_VCC1.2, R6.1, R7.2
- removed net I2C2_VCC: I2C2.1, JP_I2C2_VCC1.2, R8.1, R9.2
- removed net IC2_I0: IC2.I0, JP2_I0.2
- removed net IC2_I1: IC2.I1, JP2_I1.2
- removed net IC2_I2: IC2.I2, JP2_I2.2
- removed net IC2_I3: IC2.I3, JP2_I3.2
- removed net IC2_I4: IC2.I4, JP2_I4.2
- removed net IC2_NFAULT: IC2.NFAULT, IC2_R3.1, U$1.7
- removed net IC2_NRESET: IC2.NRESET, JP2_S.2
- removed net IC2_NSLEEP: IC2.NSLEEP, JP2_S.1
- removed net IC2_V3P3: IC2.DECAY, IC2.V3P3OUT, IC2_C6.1, IC2_R1.1, IC2_R3.2
- removed net IC3_I0: IC3.I0, JP3_I0.2
- removed net IC3_I1: IC3.I1, JP3_I1.2
- removed net IC3_I2: IC3.I2, JP3_I2.2
- removed net IC3_I3: IC3.I3, JP3_I3.2
- removed net IC3_I4: IC3.I4, JP3_I4.2
- removed net IC3_NFAULT: IC3.NFAULT, IC3_R3.1, U$1.10/CS
- removed net IC3_NRESET: IC3.NRESET, JP3_S.2
- removed net IC3_NSLEEP: IC3.NSLEEP, JP3_S.1
- removed net IC3_R2: IC3.VREF(1), IC3.VREF(2), IC3_R1.2, IC3_R2.2
- removed net IC3_V3P3: IC3.DECAY, IC3.V3P3OUT, IC3_C6.1, IC3_R1.1, IC3_R3.2
- removed net M2_1: IC2.OUT1(1), IC2.OUT1(2), M2-1.KL
- removed net M2_2: IC2.OUT2(1), IC2.OUT2(2), M2-2.KL
- removed net M3_1: IC3.OUT1(1), IC3.OUT1(2), M3-1.KL
- removed net M3_2: IC3.OUT2(1), IC3.OUT2(2), M3-2.KL
- removed net MOT2_DIR: IC2.PHASE, U$1.8
- removed net MOT2_PWM: IC2.ENBL, U$1.9/CS
- removed net MOT3_DIR: IC3.PHASE, U$1.29
- removed net MOT3_PWM: IC3.ENBL, U$1.30
- removed net N$1: JP11.4, U$1.23/A9
- removed net N$13: IC2.CP2(1), IC2_C1.1
- removed net N$14: IC2.CP2(2), IC2_C1.2
- removed net N$15: IC2.VCP, IC2_C2.2, IC2_R5.2
- removed net N$17: IC3.ISEN(1), IC3.ISEN(2), IC3_R4.2
- removed net N$18: IC3.CP2(1), IC3_C1.1
- removed net N$19: IC3.CP2(2), IC3_C1.2
- removed net N$20: IC3.VCP, IC3_C2.2, IC3_R5.2
- removed net N$3: IC2.VREF(1), IC2.VREF(2), IC2_R1.2, IC2_R2.2
- removed net N$4: JP11.3, U$1.22/A8
- removed net N$52: JP7.1, U$1.A22/DAC1
- removed net N$53: JP7.2, U$1.A21/DAC0
- removed net N$57: J1.1, U$1.36/A17
- removed net N$58: J1.2, U$1.35/A16
- removed net N$6: JP11.2, U$1.21/A7
- removed net N$7: JP12.1, U$1.11/MOSI
- removed net N$8: BAT_1-1.KL, D24V22F3.VIN, D24V50F5.VIN
- removed net N$9: IC2.ISEN(1), IC2.ISEN(2), IC2_R4.2
- removed net NS50: JP7.3, U$1.39/A20
- removed net RX1: JP_UART1.2, U$1.0/RX
- removed net RX4: JP_UART4.2, U$1.31/A12
- removed net RX5: JP_UART5.3, U$1.34/A15
- removed net SCL0: I2C0.3, R4.2, U$1.19/A5/SCL
- removed net SCL1: I2C1.3, R6.2, U$1.37/A18
- removed net SCL2: I2C2.3, R8.2, U$1.3/CANTX
- removed net SDA0: I2C0.4, R5.1, U$1.18/A4/SDA
- removed net SDA1: I2C1.4, R7.1, U$1.38/A19
- removed net SDA2: I2C2.4, R9.1, U$1.4/CANRX
- removed net TX1: JP_UART1.3, U$1.1/TX
- removed net TX4: JP_UART4.3, U$1.32/A13
- removed net TX5: JP_UART5.2, U$1.33/A14
- new net DECAY: IC1.DECAY, JP2.4
- net 12V2: no longer 12V_PWR_1-1.KL, 12V_PWR_2-1.KL, 12V_PWR_3-1.KL, BAT_2-1.KL, IC2.VM(1), IC2.VM(2), IC2_C2.1, IC2_C3.2, IC2_C4.2, IC2_C5.+, IC2_R5.1, IC3.VM(1), IC3.VM(2), IC3_C2.1, IC3_C3.2, IC3_C4.2, IC3_C5.+, IC3_R5.1
- net GND: now also JP1.1, JP2.1, JP3.1; no longer 12V_PWR_1-2.KL, 12V_PWR_2-2.KL, 12V_PWR_3-2.KL, BAT_1-2.KL, BAT_2-2.KL, D24V22F3.GND, D24V22F3.GND_2, D24V22F3.PG, D24V50F5.GND, D24V50F5.GND_2, I2C0.2, I2C1.2, I2C2.2, IC2.GND(1), IC2.GND(2), IC2.THERMAL_PAD, IC2_C3.1, IC2_C4.1, IC2_C5.-, IC2_C6.2, IC2_R2.1, IC2_R4.1, IC3.GND(1), IC3.GND(2), IC3.THERMAL_PAD, IC3_C3.1, IC3_C4.1, IC3_C5.-, IC3_C6.2, IC3_R2.1, IC3_R4.1, JP_3V3.2, JP_3V3.4, JP_3V3.6, JP_3V3.8, JP_5V.2, JP_5V.4, JP_5V.6, JP_5V.8, JP_ENC1.1, JP_ENC2.1, JP_ENC3.1, JP_UART1.4, JP_UART4.4, JP_UART5.1, U$1.AGND, U$1.GND, U$1.GND2, X_3V3-2.KL, X_3V3-4.KL, X_5V-2.KL, X_5V-4.KL, X_5V-6.KL
- net IC1_I0: now also JP1.6; no longer JP1_I0.2
- net IC1_I1: now also JP1.5; no longer JP1_I1.2
- net IC1_I2: now also JP1.4; no longer JP1_I2.2
- net IC1_I3: now also JP1.3; no longer JP1_I3.2
- net IC1_I4: now also JP1.2; no longer JP1_I4.2
- net IC1_NFAULT: no longer U$1.2
- net IC1_NRESET: now also JP3.3; no longer JP1_S.2
- net IC1_NSLEEP: now also JP3.2; no longer JP1_S.1
- net IC1_V3P3: no longer IC1.DECAY
- net MOT1_DIR: now also JP2.3; no longer U$1.5
- net MOT1_PWM: now also JP2.2; no longer U$1.6
Other:
- moved on the sheet: IC1, IC1_C1, IC1_C2, IC1_C3, IC1_C4, IC1_C5, IC1_C6, IC1_R1, IC1_R2, IC1_R3, IC1_R4, IC1_R5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
