File: 2023/CarteAlimV2/CarteDAllim.kicad_pcb (KiCad board)
At the start: 2 copper layers, 75 x 65 mm, 15 parts, among them J1 USB_A, J10 Screw_Terminal_01x02, J2 Screw_Terminal_01x02, J3 Screw_Terminal_01x02, J4 Screw_Terminal_01x02, J5 Screw_Terminal_01x02, J6 Screw_Terminal_01x02, J7 Screw_Terminal_01x02, J8 Screw_Terminal_01x02, J9 Screw_Terminal_01x02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

Commit message: CarteAlimV2-Suite et fin
Parts:
- added G***: LOGO, Logos:EnacRobotique25mm, F.Cu at (70.7, 61.7)
- added G***: LOGO, Logos:EnacRobotique50mm, B.Cu at (58.4, 63.1)
- moved REF** 5.00 mm to (95.0, 35.0)
- moved REF** 5.00 mm to (30.0, 35.0)
Other:
- board text added: "+18V"
- board text added: "+5V"
- board text added: "Arrêt Urgence"
- board text added: "GND"

Commit message: Update
Parts:
- moved G*** 0.81 mm to (70.6, 62.5)
Routing:
- net unconnected-(J1-Pad5): track 0.00 -> 13.1 mm
Changed lines of the file:
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@@
   )
   (footprint "Logos:EnacRobotique25mm" (layer "F.Cu")
-    (at 70.7136 61.6966 90)
+    (at 70.6 62.5 90)
     (attr board_only exclude_from_pos_files exclude_from_bom)
-    (fp_text reference "G***" (at 0 0 90) (layer "F.SilkS")
+    (fp_text reference "G***" (at -2.0034 0.6864 90) (layer "F.SilkS")
       (effects (font (size 1.524 1.524) (thickness 0.3)))
     )
@@
       (effects (font (size 1 1) (thickness 0.15)))
     )
-    (fp_text value "Screw_Terminal_01x02" (at 2.5 7.5 90) (layer "F.Fab")
+    (fp_text value "Screw_Terminal_01x02" (at 0.4 7.6 90) (layer "F.Fab")
       (effects (font (size 1 1) (thickness 0.15)))
     )
@@
   (segment (start 55.08 52.8) (end 48.17 45.89) (width 2) (layer "F.Cu") (net 1))
   (segment (start 55.08 52.8) (end 55.08 44.0816) (width 2) (layer "F.Cu") (net 1))
-  (segment (start 32.7914 55.88) (end 38.1 55.88) (width 5) (layer "F.Cu") (net 6))
-  (segment (start 38.1 71.12) (end 34.4932 71.12) (width 5) (layer "F.Cu") (net 6))
+  (segment (start 51.24 43.18) (end 38.1 43.18) (width 2) (layer "F.Cu") (net 5))
+  (segment (start 30.3 67) (end 32.72 69.42) (width 10) (layer "F.Cu") (net 6))
+  (segment (start 38.1 71.12) (end 34.42 71.12) (width 5) (layer "F.Cu") (net 6))
+  (segment (start 34.42 71.12) (end 32.72 69.42) (width 5) (layer "F.Cu") (net 6))
+  (segment (start 38.1 55.88) (end 33.42 55.88) (width 5) (layer "F.Cu") (net 6))
   (segment (start 38.1 55.88) (end 45.88 55.88) (width 2) (layer "F.Cu") (net 6))
-  (segment (start 34.4932 71.12) (end 30.5054 67.1322) (width 5) (layer "F.Cu") (net 6))
   (segment (start 45.88 55.88) (end 50 60) (width 2) (layer "F.Cu") (net 6))
-  (segment (start 30.5054 67.1322) (end 30.5054 58.166) (width 5) (layer "F.Cu") (net 6))
-  (segment (start 30.5054 58.166) (end 32.7914 55.88) (width 5) (layer "F.Cu") (net 6))
+  (segment (start 30.3 59) (end 30.3 67) (width 10) (layer "F.Cu") (net 6))
+  (segment (start 33.42 55.88) (end 30.3 59) (width 2) (layer "F.Cu") (net 6))
   (zone (net 7) (net_name "18V-Safe") (layer "F.Cu") (hatch edge 0.508)
     (connect_pads (clearance 0.508))
