File: 2020/robotA_2020/robotA_2020.kicad_pcb (KiCad board)
At the start: 2 copper layers, 87 x 78 mm, 38 parts, among them U1 PCA9554D, U2 NUCLEO32-L432KC, U3 PCA9554D, U4 LM2596_module, U5 IRLML6344, U6 IRLML6344, U7 IRLML6344, U8 IRLML6344, U9 IRLML6344

Commit message: update
Other:
- net class Default removed
