File: 2023/CarteAlimV2.5/CarteAlim.kicad_sch (KiCad schematic)
At the start: 13 parts, among them J1 Screw_Terminal_01x02, J10 Screw_Terminal_01x02, J11 USB_A, J12 Screw_Terminal_01x02, J2 Screw_Terminal_01x02, J3 Screw_Terminal_01x02, J4 Screw_Terminal_01x02, J5 Screw_Terminal_01x02, J6 Screw_Terminal_01x02, J7 Screw_Terminal_01x02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

Commit message: Update finale
Parts:
- removed J10, J7: Screw_Terminal_01x02, TerminalBlock:TerminalBlock_bornier-2_P5.08mm, symbol Connector:Screw_Terminal_01x02
Connections:
- net +18V is gone; now on net +18V_Bat: J8.1 (Pin_1)
Changed lines of the file:
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@@
   (no_connect (at 72.39 102.87))
   (no_connect (at 62.23 110.49))
-  (global_label "+18V_Bat" (shape input) (at 24.13 41.91 0) (fields_autoplaced)
-    (effects (font (size 1.27 1.27)) (justify left))
-    (property "Références Inter-Feuilles" "${INTERSHEET_REFS}" (id 0) (at 35.7355 41.8306 0)
-      (effects (font (size 1.27 1.27)) (justify left) hide)
-    )
-  )
   (global_label "+18V_Bat" (shape input) (at 24.13 21.59 0) (fields_autoplaced)
     (effects (font (size 1.27 1.27)) (justify left))
@@
     )
   )
-  (global_label "+18V" (shape input) (at 24.13 39.37 0) (fields_autoplaced)
-    (effects (font (size 1.27 1.27)) (justify left))
-    (property "Références Inter-Feuilles" "${INTERSHEET_REFS}" (id 0) (at 31.6231 39.2906 0)
-      (effects (font (size 1.27 1.27)) (justify left) hide)
-    )
-  )
   (global_label "+18V_prot" (shape input) (at 22.86 116.84 0) (fields_autoplaced)
     (effects (font (size 1.27 1.27)) (justify left))
@@
     )
   )
-  (global_label "+18V" (shape input) (at 24.13 57.15 0) (fields_autoplaced)
-    (effects (font (size 1.27 1.27)) (justify left))
-    (property "Références Inter-Feuilles" "${INTERSHEET_REFS}" (id 0) (at 31.6231 57.0706 0)
+  (global_label "+18V_Bat" (shape input) (at 24.13 57.15 0) (fields_autoplaced)
+    (effects (font (size 1.27 1.27)) (justify left))
+    (property "Références Inter-Feuilles" "${INTERSHEET_REFS}" (id 0) (at 35.7355 57.0706 0)
       (effects (font (size 1.27 1.27)) (justify left) hide)
     )
@@
     (effects (font (size 1.27 1.27)) (justify left))
     (property "Références Inter-Feuilles" "${INTERSHEET_REFS}" (id 0) (at 35.1307 83.7406 0)
-      (effects (font (size 1.27 1.27)) (justify left) hide)
-    )
-  )
-  (global_label "+18V" (shape input) (at 59.69 41.91 0) (fields_autoplaced)
-    (effects (font (size 1.27 1.27)) (justify left))
-    (property "Références Inter-Feuilles" "${INTERSHEET_REFS}" (id 0) (at 67.1831 41.8306 0)
       (effects (font (size 1.27 1.27)) (justify left) hide)
     )
@@
     (pin "1")
   )
-  (symbol (lib_id "power:GND") (at 59.69 39.37 90) (unit 1)
-    (in_bom yes) (on_board yes) (fields_autoplaced)
-    (property "Reference" "#PWR08" (id 0) (at 66.04 39.37 0)
-      (effects (font (size 1.27 1.27)) hide)
-    )
-    (property "Value" "GND" (id 1) (at 63.5 39.3699 90)
-      (effects (font (size 1.27 1.27)) (justify right))
-    )
-    (property "Footprint" "" (id 2) (at 59.69 39.37 0)
-      (effects (font (size 1.27 1.27)) hide)
-    )
-    (property "Datasheet" "" (id 3) (at 59.69 39.37 0)
-      (effects (font (size 1.27 1.27)) hide)
-    )
-    (pin "1")
-  )
-  (symbol (lib_id "Connector:Screw_Terminal_01x02") (at 54.61 41.91 180) (unit 1)
-    (in_bom yes) (on_board yes) (fields_autoplaced)
-    (property "Reference" "J10" (id 0) (at 54.61 35.56 0))
-    (property "Value" "Screw_Terminal_01x02" (id 1) (at 54.61 35.56 0)
-      (effects (font (size 1.27 1.27)) hide)
-    )
-    (property "Footprint" "TerminalBlock:TerminalBlock_bornier-2_P5.08mm" (id 2) (at 54.61 41.91 0)
-      (effects (font (size 1.27 1.27)) hide)
-    )
-    (property "Datasheet" "~" (id 3) (at 54.61 41.91 0)
-      (effects (font (size 1.27 1.27)) hide)
-    )
-    (pin "1")
-    (pin "2")
-  )
   (symbol (lib_id "Connector:USB_A") (at 64.77 100.33 0) (unit 1)
     (in_bom yes) (on_board yes) (fields_autoplaced)
@@
     (pin "4")
     (pin "5")
-  )
-  (symbol (lib_id "Connector:Screw_Terminal_01x02") (at 19.05 41.91 180) (unit 1)
-    (in_bom yes) (on_board yes) (fields_autoplaced)
-    (property "Reference" "J7" (id 0) (at 19.05 35.56 0))
-    (property "Value" "Screw_Terminal_01x02" (id 1) (at 19.05 35.56 0)
-      (effects (font (size 1.27 1.27)) hide)
-    )
-    (property "Footprint" "TerminalBlock:TerminalBlock_bornier-2_P5.08mm" (id 2) (at 19.05 41.91 0)
-      (effects (font (size 1.27 1.27)) hide)
-    )
-    (property "Datasheet" "~" (id 3) (at 19.05 41.91 0)
-      (effects (font (size 1.27 1.27)) hide)
-    )
-    (pin "1")
-    (pin "2")
   )
   (symbol (lib_id "power:GND") (at 24.13 69.85 90) (unit 1)
@@
       (reference "#PWR07") (unit 1) (value "GND") (footprint "")
     )
-    (path "/1f6fa88e-8fe1-4ebe-ab1d-59d4cfcaf6f9"
-      (reference "#PWR08") (unit 1) (value "GND") (footprint "")
-    )
     (path "/60d2ae6c-2809-44e7-b77e-05ced2e81f1e"
       (reference "#PWR09") (unit 1) (value "GND") (footprint "")
@@
       (reference "J6") (unit 1) (value "Screw_Terminal_01x02") (footprint "TerminalBlock:TerminalBlock_bornier-2_P5.08mm")
     )
-    (path "/5d5b044d-79b5-4215-a451-e190d70d5fd4"
-      (reference "J7") (unit 1) (value "Screw_Terminal_01x02") (footprint "TerminalBlock:TerminalBlock_bornier-2_P5.08mm")
-    )
     (path "/70f2caa4-a4ee-4e96-9dd4-1edfae4c2f0c"
       (reference "J8") (unit 1) (value "Screw_Terminal_01x02") (footprint "TerminalBlock:TerminalBlock_bornier-2_P5.08mm")
@@
       (reference "J9") (unit 1) (value "Screw_Terminal_01x02") (footprint "TerminalBlock:TerminalBlock_bornier-2_P5.08mm")
     )
-    (path "/2fa186f0-78e4-44ff-a1cf-f43e70043e11"
-      (reference "J10") (unit 1) (value "Screw_Terminal_01x02") (footprint "TerminalBlock:TerminalBlock_bornier-2_P5.08mm")
-    )
     (path "/482a4633-0447-43ed-b245-dde6fd468a30"
