File: 2023/CarteAlimV2.5/CarteAlim.kicad_pcb (KiCad board)
At the start: 2 copper layers, 70 x 60 mm, 18 parts, among them J1 Screw_Terminal_01x02, J11 USB_A, J12 Screw_Terminal_01x02, J2 Screw_Terminal_01x02, J3 Screw_Terminal_01x02, J4 Screw_Terminal_01x02, J5 Screw_Terminal_01x02, J6 Screw_Terminal_01x02, J9 Screw_Terminal_01x02, U1 TSR_1-2450

Commit message: Update finale
Parts:
- removed ESC, Fusible, J6: Screw_Terminal_01x02, TerminalBlock:TerminalBlock_bornier-2_P5.08mm
- removed the G*** at (116.8, 106.7)
- removed the REF** at (140.0, 125.0)
- removed the REF** at (80.0, 125.0)
- removed the REF** at (79.8, 75.0)
- added Batterie: Screw_Terminal_01x02, TerminalBlock:TerminalBlock_bornier-2_P5.08mm, F.Cu at (80.0, 83.8)
- added G***: LOGO, lib:logo, F.Cu at (124.5, 94.0)
- added REF**: MountingHole_3.2mm_M3, MountingHole:MountingHole_3.2mm_M3, F.Cu at (140.0, 115.0)
- added REF**: MountingHole_3.2mm_M3, MountingHole:MountingHole_3.2mm_M3, F.Cu at (80.0, 75.0)
- added REF**: MountingHole_3.2mm_M3, MountingHole:MountingHole_3.2mm_M3, F.Cu at (80.0, 115.0)
- moved J5 54.4 mm to (130.6, 74.9), turned to 180 degrees
- moved J2 46.9 mm to (94.0, 114.3), turned to 0 degrees
- moved J3 39.1 mm to (110.0, 114.3), turned to 0 degrees
- moved J9 16.5 mm to (139.7, 88.9), turned to 90 degrees
- moved J4 12.7 mm to (139.7, 104.1)
- moved J1 11.0 mm to (127.0, 114.3)
- moved Arrêt Urgence 2.79 mm to (80.1, 101.6)
- moved U1 1.70 mm to (95.7, 98.8)
- moved J11 1.37 mm to (97.5, 84.1)
- moved J12 1.28 mm to (116.2, 74.9)
Connections:
- Arrêt Urgence pad 2: +18V -> +18V_prot
Routing:
- net +5V: track 37.2 -> 0.00 mm
- net +18V_Bat: track 12.7 -> 0.00 mm
- net unconnected-(J11-Pad5): track 16.2 -> 13.1 mm
- added copper zone on F.Cu, net +5V
- removed copper zone on F.Cu, net +18V
Other:
- board size 70 x 60 mm -> 70 x 50 mm
- board text added: "+18V Batt"
- board text removed: "18V Batt"

Commit message: Fin de l'elec
Parts:
- moved J12 3.94 mm to (112.3, 74.8)
Changed lines of the file:
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@@
   )
   (footprint "TerminalBlock:TerminalBlock_bornier-2_P5.08mm" (layer "F.Cu")
-    (at 116.205 74.93 180)
+    (at 112.268 74.803 180)
     (descr "simple 2-pin terminal block, pitch 5.08mm, revamped version of bornier2")
     (tags "terminal block bornier2")
@@
   )
   (gr_rect (start 101.6 109.22) (end 111.76 83.82) (layer "F.SilkS") (width 0.15) (fill none))
+  (gr_rect (start 102.362 70.612) (end 117.729 80.264) (layer "F.SilkS") (width 0.15) (fill none))
   (gr_rect (start 75 70) (end 145 120) (layer "Edge.Cuts") (width 0.15) (fill none))
   (gr_text "GND" (at 139.827 80.391) (layer "F.SilkS")
     (effects (font (size 1 1) (thickness 0.15)))
   )
-  (gr_text "+5V" (at 119.761 75.057 90) (layer "F.SilkS")
+  (gr_text "+5V" (at 116.332 74.422 90) (layer "F.SilkS")
     (effects (font (size 1 1) (thickness 0.15)))
   )
@@
     (effects (font (size 1 1) (thickness 0.15)))
   )
-  (gr_text "GND" (at 107.569 74.803 90) (layer "F.SilkS")
+  (gr_text "GND" (at 103.251 74.295 90) (layer "F.SilkS")
     (effects (font (size 1 1) (thickness 0.15)))
   )
