File: 2023/CartePrincipaleRobot/CartePrincipaleRobot.kicad_pcb (KiCad board)
At the start: 2 copper layers, 43 parts, among them J1 Conn_01x02_Male, J10 Conn_01x03_Male, J11 Conn_01x03_Male, J12 Conn_01x03_Male, J13 Conn_01x03_Male, J14 Conn_01x03_Male, J15 Screw_Terminal_01x02, J16 Screw_Terminal_01x02, J17 Screw_Terminal_01x02, J18 Conn_01x04_Male, J19 Conn_01x04_Male, J2 Conn_01x02_Male, J20 Conn_01x02_Male, J21 Conn_01x02_Male, J22 Conn_01x02_Male, J23 Conn_01x04_Male, J24 Conn_01x04_Male, J25 Conn_01x04_Male, J26 Conn_01x04_Male, J27 Conn_01x04_Male, J28 Conn_01x04_Male, J3 Conn_01x03_Male, J4 Conn_01x03_Male, J5 Conn_01x03_Male, J6 Conn_01x03_Male, J7 Conn_01x03_Male, J8 Conn_01x03_Male, J9 Conn_01x03_Male, U1 TSR_1-2450, U2 NUCLEO-F476RG

Commit message: update
Parts:
- moved U2 51.0 mm to (55.9, 63.5)
- moved A1 27.9 mm to (118.1, 74.9), turned to 90 degrees
- moved A2 20.7 mm to (121.9, 43.2), turned to 90 degrees

Commit message: update
Parts:
- removed J1, J2, J20, J21, J22: Conn_01x02_Male, library:HE14_EMBASE_1x02
- removed J12, J13: Conn_01x03_Male, library:HE14_EMBASE_1x03
- removed J17: Screw_Terminal_01x02, TerminalBlock:TerminalBlock_bornier-2_P5.08mm
- removed J23, J24, J26, J27, J28: Conn_01x04_Male, library:HE14_EMBASE_1x04
- removed J3, J4, J5, J6, J7, J8: Conn_01x03_Male, Connector_PinSocket_2.54mm:PinSocket_1x03_P2.54mm_Vertical
- added Color: Conn_01x02_Male, library:HE14_EMBASE_1x02, F.Cu at (58.0, 35.3)
- added D1: DIODE, Diode_THT:D_A-405_P7.62mm_Horizontal, F.Cu at (61.5, 67.6)
- added D2: DIODE, Diode_THT:D_A-405_P7.62mm_Horizontal, F.Cu at (69.1, 54.6)
- added ESC: Conn_01x03_Male, Connector_PinSocket_2.54mm:PinSocket_1x03_P2.54mm_Vertical, F.Cu at (132.1, 81.8)
- added Enc1: Conn_01x04_Male, library:HE14_EMBASE_1x04, F.Cu at (96.2, 116.8)
- added Enc2: Conn_01x04_Male, library:HE14_EMBASE_1x04, F.Cu at (113.0, 116.8)
- added Enc3: Conn_01x04_Male, library:HE14_EMBASE_1x04, F.Cu at (46.0, 35.6)
- added FC1: Conn_01x02_Male, library:HE14_EMBASE_1x02, F.Cu at (62.7, 117.1)
- added FC2: Conn_01x02_Male, library:HE14_EMBASE_1x02, F.Cu at (73.2, 117.1)
- added I2C: Conn_01x04_Male, library:HE14_EMBASE_1x04, F.Cu at (87.7, 36.3)
- added I2C: Conn_01x04_Male, library:HE14_EMBASE_1x04, F.Cu at (96.4, 36.3)
- added Mot1: Conn_01x03_Male, library:HE14_EMBASE_1x03, F.Cu at (117.7, 36.4)
- added Mot2: Conn_01x03_Male, library:HE14_EMBASE_1x03, F.Cu at (110.6, 36.1)
- added PosButton: Conn_01x02_Male, library:HE14_EMBASE_1x02, F.Cu at (65.3, 35.3)
- added REF**: MountingHole_3.2mm_M3, MountingHole:MountingHole_3.2mm_M3, F.Cu at (180.0, 30.0)
- added REF**: MountingHole_3.2mm_M3, MountingHole:MountingHole_3.2mm_M3, F.Cu at (180.0, 120.0)
- added REF**: MountingHole_3.2mm_M3, MountingHole:MountingHole_3.2mm_M3, F.Cu at (40.0, 120.0)
- added REF**: MountingHole_3.2mm_M3, MountingHole:MountingHole_3.2mm_M3, F.Cu at (40.0, 30.0)
- added S1: Conn_01x03_Male, Connector_PinSocket_2.54mm:PinSocket_1x03_P2.54mm_Vertical, F.Cu at (132.3, 114.6)
- added S2: Conn_01x03_Male, Connector_PinSocket_2.54mm:PinSocket_1x03_P2.54mm_Vertical, F.Cu at (132.3, 108.0)
- added S3: Conn_01x03_Male, Connector_PinSocket_2.54mm:PinSocket_1x03_P2.54mm_Vertical, F.Cu at (132.1, 100.6)
- added S4: Conn_01x03_Male, Connector_PinSocket_2.54mm:PinSocket_1x03_P2.54mm_Vertical, F.Cu at (132.1, 93.7)
- added S5: Conn_01x03_Male, Connector_PinSocket_2.54mm:PinSocket_1x03_P2.54mm_Vertical, F.Cu at (132.1, 87.6)
- added Tir: Conn_01x02_Male, library:HE14_EMBASE_1x02, F.Cu at (55.1, 116.6)
- added U3: LM2596, library:LM2596, F.Cu at (161.5, 46.2)
- moved Afficheur 95.0 mm to (73.8, 35.4)
- moved Mot3 94.4 mm to (103.7, 36.1), turned to 90 degrees
- moved R1 87.0 mm to (111.5, 53.1), turned to 90 degrees
- moved U1 84.0 mm to (134.6, 70.5), turned to 180 degrees
- moved R3 83.1 mm to (102.9, 53.1), turned to 90 degrees
- moved R2 83.0 mm to (107.2, 53.1), turned to 90 degrees
- moved A2 78.2 mm to (178.3, 97.3), turned to -90 degrees
- moved C2 72.0 mm to (152.9, 101.2), turned to -90 degrees
- moved JP3 67.4 mm to (168.1, 76.7), turned to -90 degrees
- moved A1 60.5 mm to (178.2, 67.8), turned to -90 degrees
- moved J16 60.1 mm to (147.8, 118.9), turned to 180 degrees
- moved JP6 54.6 mm to (169.2, 104.6), turned to -90 degrees
- moved J15 46.9 mm to (128.3, 31.8)
- moved J10 44.6 mm to (131.0, 57.9), turned to 180 degrees
- moved JP4 43.6 mm to (163.1, 104.6), turned to -90 degrees
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- renumbered J25 to Afficheur, J14 to Mot3
Connections:
- U2 pad 18: 5V_Logic -> Net-(D1-Pad2)
- U2 pad 46: 5V_Logic -> Net-(D2-Pad1)
- U2 pad 6: 5V_Logic -> Net-(D1-Pad2)
Other:
- board outline added: 150 x 100 mm
- board text added: "+18V"
- board text added: "+5V"
- board text added: "GND"

Commit message: update
Parts:
- added G***: LOGO, library:logo, F.Cu at (90.7, 72.4)
- added G***: LOGO, library:logo, B.Cu at (90.4, 75.2)
- moved ESC 32.8 mm to (132.1, 114.6)
- moved S5 7.11 mm to (132.1, 80.5)
- moved S2 6.61 mm to (132.1, 101.3)
- moved S4 6.60 mm to (132.1, 87.1)
- moved S1 6.36 mm to (132.1, 108.2)
- moved S3 6.35 mm to (132.1, 94.2)
Routing:
- net 5V_Logic: track 0.00 -> 259.0 mm
- net +18V: track 0.00 -> 122.5 mm
- net ESC_PWM: track 0.00 -> 85.9 mm
- net +3.3V: track 0.00 -> 79.7 mm, vias 0 -> 1
- net Servo1: track 0.00 -> 78.5 mm
- net +5V: track 0.00 -> 78.0 mm
- net Tirette: track 0.00 -> 69.1 mm, vias 0 -> 2
- net Net-(D1-Pad2): track 0.00 -> 61.7 mm, vias 0 -> 2
- net Stepper1_FinCourse: track 0.00 -> 55.2 mm
- net Signal_AX12A: track 0.00 -> 39.4 mm
- net +12V: track 0.00 -> 34.0 mm
- net Net-(D2-Pad1): track 0.00 -> 30.0 mm
- net MOT1_DIR: track 0.00 -> 26.4 mm
- net MOT2_DIR: track 0.00 -> 25.9 mm
- net Enc3_A: track 0.00 -> 23.6 mm
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
Commit message: update
Parts:
- renumbered FC2 to J1, Mot1 to J12, Mot2 to J13, Mot3 to J14, FC1 to J2, Color to J20, PosButton to J21, Tir to J22, I2C to J23, I2C to J24, Afficheur to J25, Enc1 to J26, Enc2 to J27, Enc3 to J28, ESC to J3, S1 to J4, S2 to J5, S3 to J6, S4 to J7, S5 to J8
Routing:
- net +3.3V: track 79.7 -> 200.7 mm, vias 1 -> 9
- net Stepper1_STP: track 0.00 -> 115.8 mm, vias 0 -> 2
- net Stepper1_dir: track 0.00 -> 84.1 mm, vias 0 -> 6
- net Stepper2_STP: track 0.00 -> 78.1 mm
- net Stepper2_dir: track 0.00 -> 77.7 mm
- net +5V: track 78.0 -> 152.1 mm, vias 0 -> 2
- net Servo3: track 0.00 -> 66.9 mm
- net Servo2: track 0.00 -> 66.8 mm, vias 0 -> 2
- net Servo4: track 0.00 -> 61.3 mm, vias 0 -> 1
- net Servo5: track 0.00 -> 55.6 mm, vias 0 -> 1
- net GND: track 0.00 -> 46.9 mm, vias 0 -> 1
- net I2C_SDA: track 18.3 -> 63.0 mm, vias 0 -> 3
- net I2C_SCL: track 18.1 -> 41.5 mm
- net 5V_Logic: track 259.0 -> 253.7 mm
- net +12V: track 34.0 -> 29.8 mm
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- added copper zone on B.Cu, net GND
Other:
- board text added: "Carte Principale 2023 Robot 1 by V@ENAC & XD@ENAC"
- board text added: "JLCJLCJLCJLC"

Commit message: arrondis ++
Changed lines of the file:
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@@
   (arc (start 121.489787 89.231787) (mid 121.056241 88.58294) (end 120.904 87.817573) (width 0.6) (layer "F.Cu") (net 27))
   (segment (start 112.776 72.136) (end 112.776 74.93) (width 0.6) (layer "B.Cu") (net 27))
-  (segment (start 124.46 79.033068) (end 124.46 93.218) (width 0.6) (layer "F.Cu") (net 28))
+  (segment (start 124.46 79.033068) (end 124.46 92.803786) (width 0.6) (layer "F.Cu") (net 28))
   (segment (start 97.64736 59.80136) (end 110.041534 72.195534) (width 0.6) (layer "F.Cu") (net 28))
   (segment (start 95.89 45.79) (end 95.89 55.558719) (width 0.6) (layer "F.Cu") (net 28))
   (segment (start 113.577068 73.66) (end 119.086932 73.66) (width 0.6) (layer "F.Cu") (net 28))
-  (segment (start 125.476 94.234) (end 126.985 94.234) (width 0.6) (layer "F.Cu") (net 28))
+  (segment (start 126.304427 94.234) (end 126.985 94.234) (width 0.6) (layer "F.Cu") (net 28))
   (segment (start 122.622466 75.124466) (end 122.995534 75.497534) (width 0.6) (layer "F.Cu") (net 28))
-  (segment (start 124.46 93.218) (end 125.476 94.234) (width 0.6) (layer "F.Cu") (net 28))
+  (segment (start 124.752893 93.510893) (end 124.890214 93.648214) (width 0.6) (layer "F.Cu") (net 28))
+  (arc (start 124.46 92.803786) (mid 124.53612 93.186469) (end 124.752893 93.510893) (width 0.6) (layer "F.Cu") (net 28))
   (arc (start 95.89 55.558719) (mid 96.346723 57.85482) (end 97.64736 59.80136) (width 0.6) (layer "F.Cu") (net 28))
+  (arc (start 126.304427 94.234) (mid 125.53906 94.081759) (end 124.890214 93.648214) (width 0.6) (layer "F.Cu") (net 28))
   (arc (start 110.041534 72.195534) (mid 111.663651 73.279398) (end 113.577068 73.66) (width 0.6) (layer "F.Cu") (net 28))
   (arc (start 124.46 79.033068) (mid 124.079398 77.119651) (end 122.995534 75.497534) (width 0.6) (layer "F.Cu") (net 28))

Commit message: MAJ cartes elec
Changed lines of the file:
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@@
   (arc (start 132.091708 121.412) (mid 129.030241 120.803036) (end 126.434854 119.068854) (width 0.6) (layer "F.Cu") (net 21))
   (arc (start 119.126 104.460427) (mid 118.973759 103.69506) (end 118.540213 103.046213) (width 0.6) (layer "F.Cu") (net 21))
-  (segment (start 117.856 105.856) (end 117.856 109.649864) (width 0.6) (layer "F.Cu") (net 22))
+  (segment (start 117.856 106.684427) (end 117.856 109.649864) (width 0.6) (layer "F.Cu") (net 22))
   (segment (start 172.432331 115.867669) (end 178.308 109.992) (width 0.6) (layer "F.Cu") (net 22))
   (segment (start 133.467203 123.19) (end 154.754661 123.19) (width 0.6) (layer "F.Cu") (net 22))
   (segment (start 120.784932 116.720932) (end 122.860602 118.796602) (width 0.6) (layer "F.Cu") (net 22))
-  (segment (start 116.21 104.21) (end 117.856 105.856) (width 0.6) (layer "F.Cu") (net 22))
+  (segment (start 116.21 104.21) (end 117.270214 105.270214) (width 0.6) (layer "F.Cu") (net 22))
   (arc (start 133.467203 123.19) (mid 127.726952 122.048193) (end 122.860602 118.796602) (width 0.6) (layer "F.Cu") (net 22))
   (arc (start 172.432331 115.867669) (mid 164.321747 121.286988) (end 154.754661 123.19) (width 0.6) (layer "F.Cu") (net 22))
   (arc (start 117.856 109.649864) (mid 118.617205 113.476698) (end 120.784932 116.720932) (width 0.6) (layer "F.Cu") (net 22))
+  (arc (start 117.856 106.684427) (mid 117.703759 105.91906) (end 117.270214 105.270214) (width 0.6) (layer "F.Cu") (net 22))
   (segment (start 81.930466 115.629534) (end 90.81 106.75) (width 0.4) (layer "F.Cu") (net 23))
   (segment (start 76.454 117.094) (end 78.394932 117.094) (width 0.4) (layer "F.Cu") (net 23))

Commit message: Fin de l'elec
Parts:
- added REF**: KiCad-Logo2_6mm_SilkScreen, Symbol:KiCad-Logo2_6mm_SilkScreen, F.Cu at (167.6, 116.8)
- Alim 18 V: renamed from J16
- Alim 5V: renamed from J15
- Buck 18 -> 12: renamed from U3
- Enc 1: renamed from J26
- Enc 2: renamed from J27
- Enc 3: renamed from J28
- FC 1: renamed from J2
- FC 2: renamed from J1
- Mot 1: renamed from J12
- Mot 2: renamed from J13
- Mot 3: renamed from J14
- Servo 1: renamed from J4
- Servo 2: renamed from J5
- Servo 3: renamed from J6
- Servo 4: renamed from J7
- Servo 5: renamed from J8
- Stepper 1: renamed from J18
- Stepper 2: renamed from J19
- Transfo 18 -> 5: renamed from U1
- renumbered J9 to AX12, J25 to Afficheur, J20 to Color, J3 to ESC, J24 to I2C, J21 to Position, J22 to Tirette
Other:
- board text added: "-"
- board text added: "USB"
