File: 2023/CartePrincipaleRobot/CartePrincipaleRobot.kicad_pcb (KiCad board)
At the start: 2 copper layers, 150 x 100 mm, 52 parts, among them J10 Conn_01x03_Male, J11 Conn_01x03_Male, J23 Conn_01x04_Male, U2 NUCLEO-F476RG

Commit message: WARNING ENCODER 1
Other:
- board text added: "REMOVE R34 AND R36 SOLDER SB48 AND SB49"
Changed lines of the file:
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@@
     (effects (font (size 1.75 2) (thickness 0.3)))
+  )
+  (gr_text "REMOVE R34 AND R36\nSOLDER SB48 AND SB49" (at 78.105 93.091) (layer "F.SilkS")
+    (effects (font (size 3 3) (thickness 0.5)))
   )
   (gr_text "-" (at 152.4 81.28) (layer "F.SilkS")
