File: 2023/CartePrincipaleRobot/CartePrincipaleRobot.kicad_sch (KiCad schematic)
At the start: 45 parts, among them J1 Conn_01x02_Male, J10 Conn_01x03_Male, J11 Conn_01x03_Male, J12 Conn_01x03_Male, J13 Conn_01x03_Male, J14 Conn_01x03_Male, J15 Screw_Terminal_01x02, J16 Screw_Terminal_01x02, J18 Conn_01x04_Male, J19 Conn_01x04_Male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

Commit message: WARNING ENCODER 1
Other:
- note added: "FOR ENCODER 1: REMOVE R34 AND R36 SOLDER SB48 AND SB49"
Changed lines of the file:
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@@
     (effects (font (size 1.27 1.27)) (justify left bottom))
+  )
+  (text "FOR ENCODER 1:\nREMOVE R34 AND R36\nSOLDER SB48 AND SB49"
+    (at 96.52 66.04 0)
+    (effects (font (size 3 3)) (justify left bottom))
   )
   (text "Input utilisateur" (at 254 104.14 0)
