File: 2023/cartePanier/max3232id_breakout.kicad_pcb (KiCad board)
At the start: 2 copper layers, 70 x 75 mm, 21 parts, among them J1 Conn_01x04_Male, J2 Conn_01x02, J3 RJ45, J4 Conn_01x05_Male, J5 Conn_01x03_Male, U1 MAX3232, U2 DOIT-ESP32-DEVKIT-V1, U3 TSR_1-2450

Commit message: Fin de l'elec
Parts:
- added R3: A Calculer, Resistor_SMD:R_0805_2012Metric_Pad1.20x1.40mm_HandSolder, F.Cu at (86.4, 61.0)
- added ResVar: Conn_01x02_Male, Connector_PinHeader_2.54mm:PinHeader_1x02_P2.54mm_Vertical, F.Cu at (87.0, 67.2)
- renumbered J3 to AfficheurCaisse, J5 to Servo, J4 to Sound
Connections:
- U2 pad 3: unconnected-(U2-Pad3) -> MesurResVar
Routing:
- net MesurResVar: track 0.00 -> 12.3 mm
- net +3.3V: track 100.9 -> 106.1 mm
Other:
- board text added: "USB"
