File: 2023/cartePanier/max3232id_breakout.kicad_sch (KiCad schematic)
At the start: 17 parts, among them J1 Conn_01x04_Male, J2 Conn_01x02, J3 RJ45, J4 Conn_01x05_Male, J5 Conn_01x03_Male, U1 MAX3232, U2 DOIT-ESP32-DEVKIT-V1, U3 TSR_1-2450

Commit message: Fin de l'elec
Parts:
- added J6: Conn_01x02_Male, Connector_PinHeader_2.54mm:PinHeader_1x02_P2.54mm_Vertical, symbol Connector:Conn_01x02_Male
- added R3: A Calculer, Resistor_SMD:R_0805_2012Metric_Pad1.20x1.40mm_HandSolder, symbol Device:R
Connections:
- net +3.3V: now also R3.1
- net GND: now also J6.2 (Pin_2)
- net MesurResVar: now reaches U2.3 (GPIO39_ADC1-CH3_SENS-VN_RTC-GPIO3)
- net MesurResVar: now also J6.1 (Pin_1), R3.2
- no-connect marks 25 -> 24
Changed lines of the file:
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@@
   (no_connect (at 71.12 54.61))
   (no_connect (at 71.12 52.07))
-  (no_connect (at 71.12 49.53))
   (no_connect (at 118.11 57.15))
   (no_connect (at 118.11 62.23))
@@
     (stroke (width 0) (type default) (color 0 0 0 0))
   )
+  (wire (pts (xy 35.56 102.87) (xy 35.56 99.06))
+    (stroke (width 0) (type default) (color 0 0 0 0))
+  )
   (polyline (pts (xy 16.51 162.56) (xy 54.61 162.56))
     (stroke (width 0) (type default) (color 0 0 0 0))
@@
     )
   )
+  (global_label "MesurResVar" (shape input) (at 35.56 100.33 0) (fields_autoplaced)
+    (effects (font (size 1.27 1.27)) (justify left))
+    (property "Références Inter-Feuilles" "${INTERSHEET_REFS}" (id 0) (at 49.8869 100.2506 0)
+      (effects (font (size 1.27 1.27)) (justify left) hide)
+    )
+  )
   (global_label "SERVO" (shape input) (at 62.23 191.77 0) (fields_autoplaced)
     (effects (font (size 1.27 1.27)) (justify left))
@@
     )
   )
+  (global_label "MesurResVar" (shape input) (at 71.12 49.53 180) (fields_autoplaced)
+    (effects (font (size 1.27 1.27)) (justify right))
+    (property "Références Inter-Feuilles" "${INTERSHEET_REFS}" (id 0) (at 56.7931 49.6094 0)
+      (effects (font (size 1.27 1.27)) (justify right) hide)
+    )
+  )
   (global_label "RS232_OUT2" (shape input) (at 245.11 135.89 0) (fields_autoplaced)
     (effects (font (size 1.27 1.27)) (justify left))
@@
     (pin "2")
   )
+  (symbol (lib_id "power:+3.3V") (at 35.56 91.44 0) (unit 1)
+    (in_bom yes) (on_board yes) (fields_autoplaced)
+    (property "Reference" "#PWR015" (id 0) (at 35.56 95.25 0)
+      (effects (font (size 1.27 1.27)) hide)
+    )
+    (property "Value" "+3.3V" (id 1) (at 38.1 90.1699 0)
+      (effects (font (size 1.27 1.27)) (justify left))
+    )
+    (property "Footprint" "" (id 2) (at 35.56 91.44 0)
+      (effects (font (size 1.27 1.27)) hide)
+    )
+    (property "Datasheet" "" (id 3) (at 35.56 91.44 0)
+      (effects (font (size 1.27 1.27)) hide)
+    )
+    (pin "1")
+  )
   (symbol (lib_id "Jumper:SolderJumper_2_Open") (at 121.92 49.53 0) (unit 1)
     (in_bom yes) (on_board yes) (fields_autoplaced)
@@
     (pin "2")
   )
+  (symbol (lib_id "power:GND") (at 35.56 105.41 0) (unit 1)
+    (in_bom yes) (on_board yes) (fields_autoplaced)
+    (property "Reference" "#PWR016" (id 0) (at 35.56 111.76 0)
+      (effects (font (size 1.27 1.27)) hide)
+    )
+    (property "Value" "GND" (id 1) (at 38.1 106.6799 0)
+      (effects (font (size 1.27 1.27)) (justify left))
+    )
+    (property "Footprint" "" (id 2) (at 35.56 105.41 0)
+      (effects (font (size 1.27 1.27)) hide)
+    )
+    (property "Datasheet" "" (id 3) (at 35.56 105.41 0)
+      (effects (font (size 1.27 1.27)) hide)
+    )
+    (pin "1")
+  )
   (symbol (lib_id "Device:R") (at 20.32 173.99 0) (unit 1)
     (in_bom yes) (on_board yes) (fields_autoplaced)
@@
     )
     (property "Datasheet" "~" (id 3) (at 20.32 173.99 0)
+      (effects (font (size 1.27 1.27)) hide)
+    )
+    (pin "1")
+    (pin "2")
+  )
+  (symbol (lib_id "Device:R") (at 35.56 95.25 0) (unit 1)
+    (in_bom yes) (on_board yes) (fields_autoplaced)
+    (property "Reference" "R3" (id 0) (at 38.1 93.9799 0)
+      (effects (font (size 1.27 1.27)) (justify left))
+    )
+    (property "Value" "A Calculer" (id 1) (at 38.1 96.5199 0)
+      (effects (font (size 1.27 1.27)) (justify left))
+    )
+    (property "Footprint" "Resistor_SMD:R_0805_2012Metric_Pad1.20x1.40mm_HandSolder" (id 2) (at 33.782 95.25 90)
+      (effects (font (size 1.27 1.27)) hide)
+    )
+    (property "Datasheet" "~" (id 3) (at 35.56 95.25 0)
       (effects (font (size 1.27 1.27)) hide)
     )
@@
     )
     (pin "1")
+  )
+  (symbol (lib_id "Connector:Conn_01x02_Male") (at 30.48 102.87 0) (unit 1)
+    (in_bom yes) (on_board yes) (fields_autoplaced)
+    (property "Reference" "J6" (id 0) (at 31.115 100.33 0))
+    (property "Value" "Conn_01x02_Male" (id 1) (at 31.115 100.33 0)
+      (effects (font (size 1.27 1.27)) hide)
+    )
+    (property "Footprint" "Connector_PinHeader_2.54mm:PinHeader_1x02_P2.54mm_Vertical" (id 2) (at 30.48 102.87 0)
+      (effects (font (size 1.27 1.27)) hide)
+    )
+    (property "Datasheet" "~" (id 3) (at 30.48 102.87 0)
+      (effects (font (size 1.27 1.27)) hide)
+    )
+    (pin "1")
+    (pin "2")
   )
   (symbol (lib_id "Device:R") (at 33.02 173.99 0) (unit 1)
@@
       (reference "#PWR014") (unit 1) (value "+5V") (footprint "")
     )
+    (path "/1a116269-f3bb-4370-826c-a3abf5d3c404"
+      (reference "#PWR015") (unit 1) (value "+3.3V") (footprint "")
+    )
+    (path "/4dbd7516-43ae-4201-b414-c44bb79bdbcd"
+      (reference "#PWR016") (unit 1) (value "GND") (footprint "")
+    )
     (path "/30ba3aab-d12c-408d-940f-f2642ffd7609"
       (reference "#PWR0101") (unit 1) (value "+5V") (footprint "")
@@
       (reference "J5") (unit 1) (value "Conn_01x03_Male") (footprint "Connector_PinHeader_2.54mm:PinHeader_1x03_P2.54mm_Vertical")
     )
+    (path "/902ed0aa-fff4-4554-95db-737684e3ff3d"
+      (reference "J6") (unit 1) (value "Conn_01x02_Male") (footprint "Connector_PinHeader_2.54mm:PinHeader_1x02_P2.54mm_Vertical")
+    )
     (path "/22fc6622-4f77-4094-91f2-43597c0e6623"
       (reference "JP1") (unit 1) (value "SolderJumper_2_Open") (footprint "Jumper:SolderJumper-2_P1.3mm_Open_RoundedPad1.0x1.5mm")
@@
       (reference "R2") (unit 1) (value "R") (footprint "Resistor_SMD:R_0805_2012Metric_Pad1.20x1.40mm_HandSolder")
     )
+    (path "/63d59a86-5e19-4624-968d-01def9b41c3c"
+      (reference "R3") (unit 1) (value "A Calculer") (footprint "Resistor_SMD:R_0805_2012Metric_Pad1.20x1.40mm_HandSolder")
+    )
     (path "/d359b9e9-b424-4deb-ad5b-7f0fb24bee42"
