File: 2025/HubCAN/HubCAN.kicad_sch (KiCad schematic)
At the start: 6 parts, among them J1 Conn_01x03_Pin, J2 Conn_01x03_Pin, J3 Conn_01x03_Pin, J4 Conn_01x03_Pin, J5 Conn_01x03_Pin, J6 Screw_Terminal_01x02

Commit message: Hub CAN WIp
Parts:
- removed J6: Screw_Terminal_01x02, TerminalBlock:TerminalBlock_bornier-2_P5.08mm, symbol Connector:Screw_Terminal_01x02
- added H1, H2, H3, H4: MountingHole, MountingHole:MountingHole_3.2mm_M3, symbol Mechanical:MountingHole
- added J6: Conn_01x03_Pin, Connector_Molex:Molex_SPOX_5267-03A_1x03_P2.50mm_Vertical, symbol Connector:Conn_01x03_Pin
Connections:
- net GND: now also J4.3 (Pin_3), J5.3 (Pin_3), J6.3 (Pin_3); no longer J4.1 (Pin_1), J5.1 (Pin_1)
- net VIN: now also J6.2 (Pin_2)
- net CAN renamed SERIAL
- net SERIAL: now also J4.1 (Pin_1), J5.1 (Pin_1), J6.1 (Pin_1); no longer J4.3 (Pin_3), J5.3 (Pin_3)
Other:
- note added: "AX12A"
- note added: "STS3032"
