File: 2026/SPS6V-5V-5A/SPS6V-5V-5A.kicad_pcb (KiCad board)
At the start: 2 copper layers, 19 x 19 mm, 31 parts, among them IC1 LMR51450, J1 VIN, J2 GND, J3 +5V, J4 GND

Commit message: [alim 5V] remplace vias par footprint.
Parts:
- removed ? (x12): , 
- J1, J2, J3, J4: footprint Library:PAD_5x5mm -> ENAC_robotique:power_PAD_THT
- moved J3 3.57 mm to (6.60, 3.80), turned to 180 degrees
- moved J4 3.56 mm to (6.60, -3.80), turned to 0 degrees
- moved J1 3.50 mm to (-6.60, 3.80), turned to 180 degrees
- moved J2 3.50 mm to (-6.60, -3.80), turned to 0 degrees
Routing:
- net GND: vias 34 -> 31
